File: octanis_eps/v0.0_analog_shdn/octanis_eps.brd (EAGLE design)
At the start: 100 x 80 mm, 169 parts, among them IC10 OPA2333DGK, IC11 OPA2333DGK, IC12 OPA2333DGK, IC2 OPA2333DGK, IC3 OPA2333DGK, IC4 OPA2333DGK, IC5 OPA2333DGK, IC6 OPA2333DGK, IC7 OPA2333DGK, IC8 OPA2333DGK, IC9 OPA2333DGK, Q1 FC-12M

Commit message: initial prototype v0.1 of EPS PCB ready for production, BOM in process
Parts:
- removed C_ICU11: 100nF, rcl:C0603
- added R79, R80, R81: 1M, rcl:R0603
- added U$19, U$20: ADR127B, Octanis1_EPS:TSOT23-6
- C27, C28: value 22uF -> 100nF; device rcl:A/3216-18R -> rcl:C0603
- R10, R12, R39, R57, R6, R8: device rcl:R0603 -> rcl:R1206
- R77: value 50m -> 475k
- R78: value 50m -> 100k
- moved C29 539.5 mm to (40.0, 64.1), flipped to the bottom, turned to 180 degrees
- moved C26 518.5 mm to (41.9, 61.0), flipped to the bottom, turned to 180 degrees
- moved C28 510.9 mm to (15.2, 47.0), turned to 270 degrees
- moved C27 498.9 mm to (5.08, 43.2), turned to 270 degrees
- moved C31 495.8 mm to (48.3, 6.35), flipped to the bottom, turned to 90 degrees
- moved C30 488.1 mm to (38.1, 6.35), flipped to the bottom, turned to 90 degrees
- moved R78 455.9 mm to (40.6, 30.5), turned to 90 degrees
- moved C25 448.3 mm to (54.6, 12.7)
- moved R77 445.9 mm to (39.4, 25.4)
- moved R76 444.2 mm to (53.3, 24.1), turned to 270 degrees
- moved R75 432.2 mm to (49.5, 17.8)
- moved R74 429.1 mm to (54.6, 17.8)
- moved C12 423.2 mm to (5.08, 43.2), flipped to the bottom, turned to 270 degrees
- moved U$12 421.3 mm to (45.7, 36.8)
- moved R73 418.9 mm to (38.1, 17.8), turned to 180 degrees
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Connections:
- removed net N$62: C18.2
- new net N$35: C18.2, R60.2
- net EXT_PW: no longer C27.+, C28.+, C30.2, C31.2
- net GND: now also C27.1, C28.1, U$19.2, U$20.2; no longer C27.-, C28.-, C_ICU11.1
- net N$34: now also R80.2
- net N$36: now also U$11.24
- net N$75: now also R41.1
- net N$79: now also R81.2
- net N$80: now also R79.2
- net VCC: now also C27.2, C30.2, R79.1, R80.1, R81.1, U$19.3, U$20.3; no longer C_ICU11.2
- net VREF: now also C28.2, C31.2, U$19.4, U$20.4
Routing:
- net BT+: track 13.5 -> 83.1 mm, vias 2 -> 3
- net VCC: track 249.6 -> 300.3 mm, vias 3 -> 5
- net GND: track 0.00 -> 29.0 mm
- net N$77: track 0.00 -> 14.8 mm
- net N$78: track 0.00 -> 14.3 mm
- net N$75: track 0.00 -> 10.6 mm
- net EXT_PW: track 51.8 -> 58.1 mm
- net N$58: track 0.00 -> 4.00 mm
- net BT_IN: track 11.2 -> 9.88 mm
- net N$27: track 0.00 -> 0.68 mm
- net N$50: track 0.00 -> 0.59 mm
- net N$48: track 0.00 -> 0.59 mm
- added copper zone on layer 16, net GND
