File: octanis_eps/v0.1_mcu_shdn/octanis_eps_mcu_shdn.sch (EAGLE design)
At the start: 169 parts, among them IC10 OPA2333DGK, IC11 OPA2333DGK, IC12 OPA2333DGK, IC2 OPA2333DGK, IC3 OPA2333DGK, IC4 OPA2333DGK, IC5 OPA2333DGK, IC6 OPA2333DGK, IC7 OPA2333DGK, IC8 OPA2333DGK, IC9 OPA2333DGK, Q1 FC-12M

Commit message: initial prototype v0.1 of EPS PCB ready for production, BOM in process
Parts:
- removed BT_JMPR, SC_JMPR: (no value), jumper:JP4E
- removed C25, C30, C31, C_ICU11, C_ICU8: 100nF, rcl:C-EUC0603
- removed R66: 681k, rcl:R-EU_R0603
- removed R67, R73: 332k, rcl:R-EU_R0603
- removed R68: 100k, rcl:R-EU_R0603
- removed R69: 475k, rcl:R-EU_R0603
- removed R72: 825k, rcl:R-EU_R0603
- removed R74: 430, rcl:R-EU_R0603
- removed R75: 2M4, rcl:R-EU_R0603
- removed R76: 82k5, rcl:R-EU_R0603
- removed R77, R78: 50m, rcl:R-EU_R0603
- removed U$10: FDV302P, Octanis1_EPS:FDV302P
- removed U$12, U$9: FDV301N, Octanis1_EPS:FDV301N
- added R79, R80, R81: 1M, rcl:R-EU_R0603
- added U$19: ADR127B, Octanis1_EPS:ADR127B
- C27, C28: value 22uF -> 100nF; device rcl:CPOL-EUA/3216-18R -> rcl:C-EUC0603
- R10, R12, R39, R57, R6, R8: device rcl:R-EU_R0603 -> rcl:R-EU_R1206
- R46, R47: value 10k -> 100k
- R70: value 100k -> 1M
- U$8: value LTC1442 -> FDV301N; device Octanis1_EPS:LTC1442 -> Octanis1_EPS:FDV301N
Connections:
- removed net BT-: BT_IN.1, BT_IN.2, BT_JMPR.2, BT_JMPR.4, R22.2
- removed net N$66: LTC3411.SHDN/RT, R59.1, U$10.D
- removed net N$67: R66.2, R67.1, U$8.INB-
- removed net N$68: R68.2, U$8.OUTB
- removed net N$69: R68.1, R69.1, U$9.G
- removed net N$70: R72.2, R73.1, U$8.INA+
- removed net N$71: R70.2, U$10.G, U$9.D
- removed net N$72: R74.1, R76.1, U$8.REF
- removed net N$73: R75.1, R76.2, U$8.HYST
- removed net N$74: C25.2, R74.2
- removed net N$76: R77.1, R78.2, U$12.G
- removed net SC-: SC_BOT.3, SC_BOT.4, SC_JMPR.2, SC_JMPR.4, SC_TOP.3, SC_TOP.4
- removed net THD_DETECT: R78.1, U$8.OUTA
- new net EN_CHG: IC9B.+IN, U$1.29, U$8.G
- new net N$35: C18.2, R60.2
- net AEXT4: now also U$1.80; no longer U$1.6
- net A_EXT1: now also U$1.77; no longer U$1.3
- net A_EXT2: now also U$1.78; no longer U$1.4
- net A_EXT3: now also U$1.79; no longer U$1.5
- net BT+: now also LTC3411.PVIN, LTC3411.SVIN, R65.1; no longer R66.1, R72.1, U$10.S
- net EN_EXT1: now also U$1.31; no longer U$1.57
- net EN_EXT2: now also U$1.32; no longer U$1.58
- net EN_EXT3: now also U$1.33; no longer U$1.59
- net EXT_PW: no longer C27.+, C28.+, C30.2, C31.2
- net GND: now also BT_IN.1, BT_IN.2, C27.1, C28.1, R22.2, SC_BOT.3, SC_BOT.4, SC_TOP.3, SC_TOP.4, U$19.GND, U$8.S; no longer BT_JMPR.1, BT_JMPR.3, C25.1, C27.-, C28.-, C30.1, C31.1, C_ICU11.1, C_ICU8.1, IC9B.+IN, IC9B.-IN, R59.2, R67.2, R69.2, R73.2, R75.2, R77.2, SC_JMPR.1, SC_JMPR.3, U$12.S, U$8.V-, U$9.S
- net I_CHG_MS: now also U$1.7; no longer U$1.79
- net I_DSG_MS: now also U$1.8; no longer U$1.80
- net I_EXT_PW: now also U$1.6; no longer U$1.78
- net I_SC: now also U$1.5; no longer U$1.77
- net N$34: now also R80.2
- net N$36: now also U$11.VC
- net N$37: now also IC9B.-IN, IC9B.OUT; no longer U$12.D
- net N$62: now also LTC3411.SHDN/RT, R59.1; no longer C18.2
- net N$65: now also R59.2, R70.2, U$8.D; no longer LTC3411.PVIN, LTC3411.SVIN, R65.1
- net N$75: now also R41.1
- net N$79: now also R81.2
- net N$80: now also R79.2
- net VCC: now also C27.2, R79.1, R80.1, R81.1, U$19.VIN; no longer C_ICU11.2, C_ICU8.2, U$8.V+
- net VREF: now also C28.2, U$19.VOUT
Other:
- note removed: "connect BT jumper"
- note removed: "connect SC jumper"
- moved on the sheet: A_EXT, BT_IN, IC9B, JP7, R59, R70
