File: octanis_eps/v0.2_compact_version/octanis_eps_compact_no_OPA2333.sch (EAGLE design)
At the start: 90 parts, among them IC3 OPA2333DGK, IC5 OPA2333DGK, IC6 OPA2333DGK, IC7 OPA2333DGK, IC9 OPA2333DGK, Q1 FC-12M, Q2 N-HEXFET-2D_SOT232-, Q3 N-HEXFET-2D_SOT232-, Q4 N-HEXFET-2D_SOT232-

Commit message: compact version 5X6cm with MSP420Gxx24
Parts:
- removed C20: 470nF, rcl:C-EUC0603
- removed C23, C_IC3, C_IC6: 100nF, rcl:C-EUC0603
- removed IC3, IC6: OPA2333DGK, linear:OPA2333DGK
- removed R48: 1M, rcl:R-EU_R0603
- removed U$1: F552X---PN80, TI_MSP430_v16:F552X---PN80
- added U$6: MSP430G2544, Octanis1_EPS:MSP430G2544
Connections:
- removed net AEXT4: A_EXT.1, U$1.80
- removed net N$11: C6.2, IC5B.+IN, R16.1
- removed net N$27: R48.2, U$1.63
- removed net N$28: U$1.45
- removed net N$49: C20.1, U$1.20
- removed net N$6: C2.2, IC3A.+IN, R7.1
- removed net N$7: C3.2, IC3B.+IN, R9.1
- removed net N$9: C7.2, IC6B.+IN, R21.1
- new net A_EXT4: A_EXT.1, U$6.P4.6/TBOUTH/A15
- net +3V3: now also FERRITE_BEAD.1, U$6.DVCC; no longer C21.2, C23.1, FERRITE_BEAD.2, U$1.14, U$1.18, U$1.50
- net A_EXT1: now also U$6.P4.3/TB0/A12; no longer U$1.77
- net A_EXT2: now also U$6.P4.4/TB1/A13; no longer U$1.78
- net A_EXT3: now also U$6.P4.5/TB2/A14; no longer U$1.79
- net EN_CHG: now also U$6.P1.4/SMCLK/TCK; no longer U$1.29
- net EN_EXT1: now also U$6.P4.0/TB0; no longer U$1.31
- net EN_EXT2: now also U$6.P4.1/TB1; no longer U$1.32
- net EN_EXT3: now also U$6.P4.2/TB2; no longer U$1.33
- net EN_HEAT1: now also U$6.P1.1/TA0; no longer U$1.34
- net EN_HEAT2: now also U$6.P1.2/TA1; no longer U$1.35
- net EN_HEAT3: now also U$6.P1.3/TA2; no longer U$1.36
- net EXT_PW: now also U$8.A
- net GND: now also C21.1, U$6.AVSS, U$6.DVSS; no longer C20.2, C23.2, C_IC3.1, C_IC6.1, IC3P.V-, IC6P.V-, R48.1, U$1.19, U$1.49, U$1.61, U$1.68
- net I2C_SCL: now also U$6.P3.2/UCB0SOMI/UCB0SCL; no longer U$1.47
- net I2C_SDA: now also U$6.P3.1/UCB0SIMO/UCB0SDA; no longer U$1.46
- net I_EXT_PW: now also C2.2, R7.1, U$6.P2.2/TA0/A2; no longer IC3A.-IN, IC3A.OUT, U$1.6
- net I_SC: now also C3.2, R9.1, U$6.P2.1/TAINCLK/SMCLK/A1; no longer IC3B.-IN, IC3B.OUT, U$1.5
- net N$10: now also IC5B.OUT; no longer IC6A.OUT
- net N$15: now also IC5B.-IN; no longer IC6A.-IN
- net N$16: now also IC5B.+IN; no longer IC6A.+IN
- net N$48: now also U$6.XOUT/P2.7; no longer U$1.12
- net N$50: now also U$6.XIN/P2.6; no longer U$1.13
- net RST/SBWTDIO: now also U$6.RST/NMI/SBWTDIO; no longer U$1.76
- net TEST/SBWTCK: now also U$6.TEST/SBWTCK; no longer U$1.71
- net VCC: now also C21.2, FERRITE_BEAD.2, U$6.AVCC; no longer C21.1, C_IC3.2, C_IC6.2, FERRITE_BEAD.1, IC3P.V+, IC6P.V+, U$1.11, U$8.A
- net V_BT_MS: now also C7.2, R21.1, U$6.P3.7/A7; no longer IC6B.-IN, IC6B.OUT, U$1.2
- net V_BUS_MS: now also C6.2, R16.1, U$6.P3.6/A6; no longer IC5B.-IN, IC5B.OUT, U$1.1
Other:
- note removed: "DISSIPATION"
- note removed: "I2C BUS"
- moved on the sheet: A_EXT, C14, C15, C21, C22, C24, FERRITE_BEAD, IC5B, JP7, Q1

Commit message: correction & redesign on of the boost converter running
Parts:
- removed U$13, U$14, U$15: FDV301N, Octanis1_EPS:FDV301N
- removed U$8, U$9: MBRM120LTIG, Octanis1_EPS:MBRM120LTIG
- added R4: 100k, rcl:R-EU_R0603
- C2, C3, C6, C7: value 150nF -> 1.5uF
- JP1: device pinhead:PINHD-2X10 -> pinhead:PINHD-2X12
- R11: value 549k -> 50k
- R12: value 1.3M -> 286k
- R16, R21, R7, R9: value 10k -> 1k
Connections:
- removed net N$17: IC7A.-IN, IC7A.OUT
- removed net N$34: R80.2, U$15.D, U$17.EN
- removed net N$79: R81.2, U$13.D, U$16.EN
- removed net N$80: R79.2, U$14.D, U$18.EN
- net DISSIP: now also JP1.24; no longer JP1.20, U$9.A
- net EN_EXT1: now also R81.2, U$16.EN; no longer U$13.G
- net EN_EXT2: now also R80.2, U$17.EN; no longer U$15.G
- net EN_EXT3: now also R79.2, U$18.EN; no longer U$14.G
- net EXT_PW: now also JP1.18, JP1.20, JP1.22; no longer U$8.A
- net GND: now also JP1.23, Q2.S, Q3.S, Q4.S; no longer U$13.S, U$14.S, U$15.S
- net HEAT1: now also Q2.D; no longer Q2.S
- net HEAT2: now also Q3.D; no longer Q3.S
- net HEAT3: now also JP1.21, Q4.D; no longer JP1.18, Q4.S
- net N$18: no longer IC7A.+IN
- net N$23: now also R4.1
- net N$5: now also R4.2; no longer Q2.D, Q3.D, Q4.D, U$8.K, U$9.K
Other:
- moved on the sheet: C2, C27, C28, C3, C8, IC7A, Q2, R11, R6, R7, R8, R9

Commit message: completed FeedBack loop regulation on charge circuit & routing
Parts:
- added C1: 10nF, rcl:C-EUC0603
- added C_IC1: 100nF, rcl:C-EUC0603
- added IC1: OPA2333DGK, linear:OPA2333DGK
- added R30: 20k, rcl:R-EU_R0603
- added R31: 23.2k, rcl:R-EU_R0603
- added R33: 1M, rcl:R-EU_R0603
- added R34, R35, R36: 162k, rcl:R-EU_R0603
- added R37: 50m, rcl:R-EU_R1206
- added R38, R39: 10k, rcl:R-EU_R0603
- added R40, R41: 920k, rcl:R-EU_R0603
- added R5: 31.60k, rcl:R-EU_R0603
- R11: value 50k -> 100k
- R12: value 286k -> 200k
- R4: value 100k -> 560k
Connections:
- new net BT_CHG: C8.2, R12.1, R37.2, R38.1, U$10.K, U$4.VOUT
- new net CHG_CMD: C1.1, IC1B.OUT, R4.2
- new net N$11: IC1B.-IN, R34.1, R35.2, R36.2
- new net N$17: IC7A.-IN, R38.2, R41.1
- new net N$27: C1.2, R34.2
- new net N$28: IC7A.+IN, R39.2, R40.1
- new net N$6: IC1A.+IN, R30.1, R5.2
- new net N$7: IC1A.-IN, R31.1, R33.1
- new net N$9: IC1A.OUT, R33.2, R35.1
- net BT+: now also R37.1, R39.1; no longer C8.2, R12.1, U$10.K, U$4.VOUT
- net GND: now also C_IC1.1, IC1P.V-, R30.2
- net N$5: now also IC7A.OUT, R36.1, R41.2; no longer R4.2
- net VCC: now also C_IC1.2, IC1P.V+, R5.1
- net VREF: now also IC1B.+IN, R31.2, R40.2
Other:
- note added: "CHG_CMD = 3 Vref - V IC1A - V IC7A"
- note added: "Charge command"
- note added: "Command between 0 V (BT+ at 4.2V) and 2.5 V (BT+ at 3.3V)"
- note added: "Command increases when I diminishes (max 300mA limitation)"
- note added: "Command increases when VCC drops"
- note added: "IC1 : 17.09 VCC - 43.103 Vref"
- note added: "IC7: Vout = Vref - 41.6 * 0.05 * I"
- note added: "VFB is fixed at 1.25 Playing with CHG_CMD allow to tune for BT_CHG voltage between 3.3V and 4.2V"
- moved on the sheet: 10UH, C11, C4, C5, C8, IC7A, R10, R11, R12, R28, R32, R4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
