File: octanis_main_pcb_v0.1/octanis_v0.1.sch (EAGLE design)
At the start: 81 parts, among them IC1 REG1117, IC2 MPU-6050, Q1 32.768kHz, T1 BC547, T2 BC547, U1 BQ24210, U2 BQ27510_DRZ_12, U3 DRV8836DSSR, U4 DRV8836DSSR, U5 DRV8836DSSR, U6 MSP430F5529IPNR, U7 DRV8836DSSR, U9 BMP180

Commit message: created gerber files, with logo. In v0.1
Parts:
- added DIGITAL1: DIGITAL1, pinhead:PINHD-1X6
- added DIGITAL2: DIGITAL2, pinhead:PINHD-1X8
- ANALOG: value (none) -> ANALOG
- BATTERY: value (none) -> BAT
- JP2: value (none) -> SERIAL
Connections:
- new net N$14: DIGITAL2.1, U6.60
- new net N$15: DIGITAL2.2, U6.59
- new net N$20: DIGITAL2.3, U6.58
- new net N$21: DIGITAL2.4, U6.57
- new net N$22: DIGITAL2.5, U6.56
- new net N$23: DIGITAL2.6, U6.55
- new net N$24: DIGITAL2.7, U6.54
- new net N$26: DIGITAL2.8, U6.53
- net P2.7: now also DIGITAL1.6
- net P3.0: now also DIGITAL1.5
- net P3.1: now also DIGITAL1.4
- net P3.2: now also DIGITAL1.3
- net P3.3: now also DIGITAL1.2
- net P3.4: now also DIGITAL1.1
Changed lines of the file:
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@@
 <part name="TEMP1" library="varistor" deviceset="THERMISTOR" device="-2,5" value="103AT"/>
 <part name="RT1" library="resistor" deviceset="R-EU_" device="R1206" value="21.5k"/>
-<part name="BATTERY" library="pinhead" deviceset="PINHD-1X2" device=""/>
+<part name="BATTERY" library="pinhead" deviceset="PINHD-1X2" device="" value="BAT"/>
 <part name="RVDM" library="resistor" deviceset="R-EU_" device="R1206" value="float"/>
 <part name="R4" library="resistor" deviceset="R-EU_" device="R1206" value="500"/>
@@
 <part name="GND32" library="supply1" deviceset="GND" device=""/>
 <part name="I2C" library="pinhead" deviceset="PINHD-1X2" device="" value="I2C"/>
-<part name="JP2" library="pinhead" deviceset="PINHD-1X4" device=""/>
-<part name="ANALOG" library="pinhead" deviceset="PINHD-1X6" device=""/>
+<part name="JP2" library="pinhead" deviceset="PINHD-1X4" device="" value="SERIAL"/>
+<part name="ANALOG" library="pinhead" deviceset="PINHD-1X6" device="" value="ANALOG"/>
+<part name="DIGITAL1" library="pinhead" deviceset="PINHD-1X6" device="" value="DIGITAL1"/>
+<part name="DIGITAL2" library="pinhead" deviceset="PINHD-1X8" device="" value="DIGITAL2"/>
 </parts>
 <sheets>
@@
 <instance part="JP2" gate="A" x="434.34" y="167.64"/>
 <instance part="ANALOG" gate="A" x="281.94" y="261.62" rot="R180"/>
+<instance part="DIGITAL1" gate="A" x="391.16" y="157.48" rot="R270"/>
+<instance part="DIGITAL2" gate="A" x="416.56" y="241.3"/>
 </instances>
 <busses>
@@
 <net name="P3.2" class="0">
 <segment>
-<wire x1="375.92" y1="175.26" x2="375.92" y2="185.42" width="0.1524" layer="91"/>
+<wire x1="393.7" y1="160.02" x2="393.7" y2="172.72" width="0.1524" layer="91"/>
+<wire x1="393.7" y1="172.72" x2="375.92" y2="172.72" width="0.1524" layer="91"/>
+<wire x1="375.92" y1="172.72" x2="375.92" y2="185.42" width="0.1524" layer="91"/>
 <pinref part="U6" gate="G$1" pin="39"/>
 <label x="375.92" y="175.26" size="1.778" layer="95" rot="R90"/>
+<pinref part="DIGITAL1" gate="A" pin="3"/>
 </segment>
 </net>
@@
 <label x="402.59" y="203.2" size="1.778" layer="95"/>
 <wire x1="396.24" y1="203.2" x2="408.94" y2="203.2" width="0.1524" layer="91"/>
+<wire x1="408.94" y1="203.2" x2="408.94" y2="175.26" width="0.1524" layer="91"/>
+<wire x1="408.94" y1="175.26" x2="398.78" y2="175.26" width="0.1524" layer="91"/>
+<pinref part="DIGITAL1" gate="A" pin="1"/>
+<wire x1="398.78" y1="175.26" x2="398.78" y2="160.02" width="0.1524" layer="91"/>
 </segment>
 </net>
 <net name="P3.3" class="0">
 <segment>
+<wire x1="396.24" y1="160.02" x2="396.24" y2="175.26" width="0.1524" layer="91"/>
+<wire x1="396.24" y1="175.26" x2="378.46" y2="175.26" width="0.1524" layer="91"/>
 <wire x1="378.46" y1="175.26" x2="378.46" y2="185.42" width="0.1524" layer="91"/>
 <pinref part="U6" gate="G$1" pin="40"/>
 <label x="378.46" y="175.26" size="1.778" layer="95" rot="R90"/>
+<pinref part="DIGITAL1" gate="A" pin="2"/>
 </segment>
 </net>
 <net name="P2.7" class="0">
 <segment>
-<wire x1="368.3" y1="175.26" x2="368.3" y2="185.42" width="0.1524" layer="91"/>
+<wire x1="386.08" y1="160.02" x2="386.08" y2="165.1" width="0.1524" layer="91"/>
+<wire x1="386.08" y1="165.1" x2="368.3" y2="165.1" width="0.1524" layer="91"/>
+<wire x1="368.3" y1="165.1" x2="368.3" y2="185.42" width="0.1524" layer="91"/>
 <pinref part="U6" gate="G$1" pin="36"/>
 <label x="368.3" y="175.26" size="1.778" layer="95" rot="R90"/>
+<pinref part="DIGITAL1" gate="A" pin="6"/>
 </segment>
 </net>
@@
 <net name="P3.0" class="0">
 <segment>
-<wire x1="370.84" y1="175.26" x2="370.84" y2="185.42" width="0.1524" layer="91"/>
+<wire x1="388.62" y1="160.02" x2="388.62" y2="167.64" width="0.1524" layer="91"/>
+<wire x1="388.62" y1="167.64" x2="370.84" y2="167.64" width="0.1524" layer="91"/>
+<wire x1="370.84" y1="167.64" x2="370.84" y2="185.42" width="0.1524" layer="91"/>
 <pinref part="U6" gate="G$1" pin="37"/>
 <label x="370.84" y="175.26" size="1.778" layer="95" rot="R90"/>
+<pinref part="DIGITAL1" gate="A" pin="5"/>
 </segment>
 </net>
 <net name="P3.1" class="0">
 <segment>
-<wire x1="373.38" y1="175.26" x2="373.38" y2="185.42" width="0.1524" layer="91"/>
+<wire x1="391.16" y1="160.02" x2="391.16" y2="170.18" width="0.1524" layer="91"/>
+<wire x1="391.16" y1="170.18" x2="373.38" y2="170.18" width="0.1524" layer="91"/>
+<wire x1="373.38" y1="170.18" x2="373.38" y2="185.42" width="0.1524" layer="91"/>
 <pinref part="U6" gate="G$1" pin="38"/>
 <label x="373.38" y="175.26" size="1.778" layer="95" rot="R90"/>
+<pinref part="DIGITAL1" gate="A" pin="4"/>
 </segment>
 </net>
@@
 </segment>
 </net>
+<net name="N$14" class="0">
+<segment>
+<pinref part="U6" gate="G$1" pin="60"/>
+<pinref part="DIGITAL2" gate="A" pin="1"/>
+<wire x1="414.02" y1="251.46" x2="396.24" y2="251.46" width="0.1524" layer="91"/>
+</segment>
+</net>
+<net name="N$15" class="0">
+<segment>
+<pinref part="U6" gate="G$1" pin="59"/>
+<pinref part="DIGITAL2" gate="A" pin="2"/>
+<wire x1="414.02" y1="248.92" x2="396.24" y2="248.92" width="0.1524" layer="91"/>
+</segment>
+</net>
+<net name="N$20" class="0">
+<segment>
+<pinref part="U6" gate="G$1" pin="58"/>
+<pinref part="DIGITAL2" gate="A" pin="3"/>
+<wire x1="414.02" y1="246.38" x2="396.24" y2="246.38" width="0.1524" layer="91"/>
+</segment>
+</net>
+<net name="N$21" class="0">
+<segment>
+<pinref part="U6" gate="G$1" pin="57"/>
+<pinref part="DIGITAL2" gate="A" pin="4"/>
+<wire x1="414.02" y1="243.84" x2="396.24" y2="243.84" width="0.1524" layer="91"/>
+</segment>
+</net>
+<net name="N$22" class="0">
+<segment>
+<pinref part="U6" gate="G$1" pin="56"/>
+<pinref part="DIGITAL2" gate="A" pin="5"/>
+<wire x1="414.02" y1="241.3" x2="396.24" y2="241.3" width="0.1524" layer="91"/>
+</segment>
+</net>
+<net name="N$23" class="0">
+<segment>
+<pinref part="U6" gate="G$1" pin="55"/>
+<pinref part="DIGITAL2" gate="A" pin="6"/>
+<wire x1="414.02" y1="238.76" x2="396.24" y2="238.76" width="0.1524" layer="91"/>
+</segment>
+</net>
+<net name="N$24" class="0">
+<segment>
+<pinref part="U6" gate="G$1" pin="54"/>
+<pinref part="DIGITAL2" gate="A" pin="7"/>
+<wire x1="414.02" y1="236.22" x2="396.24" y2="236.22" width="0.1524" layer="91"/>
+</segment>
+</net>
+<net name="N$26" class="0">
+<segment>
+<pinref part="U6" gate="G$1" pin="53"/>
+<pinref part="DIGITAL2" gate="A" pin="8"/>
+<wire x1="414.02" y1="233.68" x2="396.24" y2="233.68" width="0.1524" layer="91"/>
+</segment>
+</net>

Commit message: corrected silk layer
Parts:
- BATTERY: value BAT -> - BAT +
- C10: value 4.7µ -> 4.7uF
- C13: value 0.22µ -> 0.22uF
- C15: value 0.1µ -> 0.1uF
- COMPASS: value HMC5883L -> HMC5883L
- HEATPAD: value 22-23-2021 -> HEATPAD
- I2C: value I2C -> SCL SDA
- JP1: value SBW -> d SBW clk
- LED3: value (none) -> 5V-ok
- RG1: value (none) -> 1.8M
- RG2: value (none) -> 18.2k
- SOLAR: value SOLAR -> - SOLAR +
- renumbered IC2 to MPU-6050
Changed lines of the file:
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@@
 <part name="TEMP1" library="varistor" deviceset="THERMISTOR" device="-2,5" value="103AT"/>
 <part name="RT1" library="resistor" deviceset="R-EU_" device="R1206" value="21.5k"/>
-<part name="BATTERY" library="pinhead" deviceset="PINHD-1X2" device="" value="BAT"/>
+<part name="BATTERY" library="pinhead" deviceset="PINHD-1X2" device="" value="-  BAT  +"/>
 <part name="RVDM" library="resistor" deviceset="R-EU_" device="R1206" value="float"/>
 <part name="R4" library="resistor" deviceset="R-EU_" device="R1206" value="500"/>
-<part name="SOLAR" library="pinhead" deviceset="PINHD-1X2" device="" value="SOLAR"/>
+<part name="SOLAR" library="pinhead" deviceset="PINHD-1X2" device="" value="- SOLAR + "/>
 <part name="U2" library="bq27510_drz_12" deviceset="BQ27510_DRZ_12" device=""/>
 <part name="C14" library="rcl" deviceset="C-EU" device="C0603" value="100n"/>
@@
 <part name="TEMP2" library="varistor" deviceset="THERMISTOR" device="-2,5" value="103AT"/>
 <part name="RSBAT" library="resistor" deviceset="R-EU_" device="R1206" value="0.01"/>
-<part name="RG2" library="rcl" deviceset="R-EU_" device="R0603"/>
-<part name="RG1" library="rcl" deviceset="R-EU_" device="R0603"/>
+<part name="RG2" library="rcl" deviceset="R-EU_" device="R0603" value="18.2k"/>
+<part name="RG1" library="rcl" deviceset="R-EU_" device="R0603" value="1.8M"/>
 <part name="RG5" library="rcl" deviceset="R-EU_" device="R0603" value="100"/>
 <part name="RG6" library="rcl" deviceset="R-EU_" device="R0603" value="100"/>
@@
 <part name="C6" library="rcl" deviceset="C-EU" device="C0603" value="22uF"/>
 <part name="SUPPLY4" library="supply2" deviceset="GND" device=""/>
-<part name="LED3" library="adafruit" deviceset="LED" device="CHIPLED_0603"/>
+<part name="LED3" library="adafruit" deviceset="LED" device="CHIPLED_0603" value="5V-ok"/>
 <part name="R6" library="rcl" deviceset="R-EU_" device="R0603" value="1k"/>
 <part name="SUPPLY7" library="supply2" deviceset="GND" device=""/>
@@
 <part name="P+1" library="supply1" deviceset="VCC" device="" value="BAT+"/>
 <part name="P+3" library="supply1" deviceset="VCC" device="" value="VCC"/>
-<part name="HEATPAD" library="con-molex" deviceset="22-23-2021" device=""/>
+<part name="HEATPAD" library="con-molex" deviceset="22-23-2021" device="" value="HEATPAD"/>
 <part name="U3" library="DRV8834" deviceset="DRV8836DSSR" device=""/>
 <part name="SV1" library="con-lstb" deviceset="MA04-1" device=""/>
@@
 <part name="GND28" library="supply1" deviceset="GND" device=""/>
 <part name="SUPPLY10" library="supply2" deviceset="+5V" device=""/>
-<part name="JP1" library="pinhead" deviceset="PINHD-1X2" device="" value="SBW"/>
+<part name="JP1" library="pinhead" deviceset="PINHD-1X2" device="" value="d SBW clk"/>
 <part name="Q1" library="crystal" deviceset="FC-12M" device="" value="32.768kHz">
 <attribute name="URL" value="http://www.mouser.ch/ProductDetail/ECS/ECS-327-125-12-TR/?qs=sGAEpiMZZMsBj6bBr9Q9adKxTNdvE4KvM1b8HDkgjuY%3d"/>
@@
 <part name="GND6" library="SparkFun-Aesthetics" deviceset="GND" device=""/>
 <part name="+3V4" library="supply1" deviceset="+3V3" device=""/>
-<part name="COMPASS" library="HMC5883L" deviceset="HMC5883L" device=""/>
+<part name="COMPASS" library="HMC5883L" deviceset="HMC5883L" device="" value="HMC5883L "/>
 <part name="GND5" library="supply1" deviceset="GND" device=""/>
 <part name="+3V5" library="supply1" deviceset="+3V3" device=""/>
-<part name="C13" library="rcl" deviceset="C-EU" device="C0603" value="0.22µ"/>
-<part name="C10" library="rcl" deviceset="C-EU" device="C0603" value="4.7µ"/>
-<part name="C15" library="rcl" deviceset="C-EU" device="C0603" value="0.1µ"/>
+<part name="C13" library="rcl" deviceset="C-EU" device="C0603" value="0.22uF"/>
+<part name="C10" library="rcl" deviceset="C-EU" device="C0603" value="4.7uF"/>
+<part name="C15" library="rcl" deviceset="C-EU" device="C0603" value="0.1uF"/>
 <part name="GND7" library="supply1" deviceset="GND" device=""/>
-<part name="IC2" library="seb" deviceset="MPU-6050" device=""/>
+<part name="MPU-6050" library="seb" deviceset="MPU-6050" device=""/>
 <part name="GND9" library="supply1" deviceset="GND" device=""/>
 <part name="GND10" library="supply1" deviceset="GND" device=""/>
@@
 <part name="+3V8" library="supply1" deviceset="+3V3" device=""/>
 <part name="GND32" library="supply1" deviceset="GND" device=""/>
-<part name="I2C" library="pinhead" deviceset="PINHD-1X2" device="" value="I2C"/>
+<part name="I2C" library="pinhead" deviceset="PINHD-1X2" device="" value="SCL SDA"/>
 <part name="JP2" library="pinhead" deviceset="PINHD-1X4" device="" value="SERIAL"/>
 <part name="ANALOG" library="pinhead" deviceset="PINHD-1X6" device="" value="ANALOG"/>
@@
 <instance part="C15" gate="G$1" x="853.44" y="292.1"/>
 <instance part="GND7" gate="1" x="883.92" y="299.72" rot="R90"/>
-<instance part="IC2" gate="G$1" x="838.2" y="137.16"/>
+<instance part="MPU-6050" gate="G$1" x="838.2" y="137.16"/>
 <instance part="GND9" gate="1" x="800.1" y="154.94" rot="R270"/>
 <instance part="GND10" gate="1" x="789.94" y="124.46" rot="R270"/>
@@
 <segment>
 <wire x1="802.64" y1="154.94" x2="805.18" y2="154.94" width="0.1524" layer="91"/>
-<pinref part="IC2" gate="G$1" pin="1"/>
+<pinref part="MPU-6050" gate="G$1" pin="1"/>
 <pinref part="GND9" gate="1" pin="GND"/>
 </segment>
 <segment>
 <wire x1="792.48" y1="124.46" x2="805.18" y2="124.46" width="0.1524" layer="91"/>
-<pinref part="IC2" gate="G$1" pin="18"/>
+<pinref part="MPU-6050" gate="G$1" pin="18"/>
 <pinref part="GND10" gate="1" pin="GND"/>
 </segment>
 <segment>
 <wire x1="792.48" y1="129.54" x2="805.18" y2="129.54" width="0.1524" layer="91"/>
-<pinref part="IC2" gate="G$1" pin="P"/>
+<pinref part="MPU-6050" gate="G$1" pin="P"/>
 <pinref part="GND12" gate="1" pin="GND"/>
 </segment>
@@
 <wire x1="866.14" y1="116.84" x2="863.6" y2="116.84" width="0.1524" layer="91"/>
 <pinref part="GND15" gate="1" pin="GND"/>
-<pinref part="IC2" gate="G$1" pin="11"/>
+<pinref part="MPU-6050" gate="G$1" pin="11"/>
 </segment>
 <segment>
 <wire x1="863.6" y1="147.32" x2="866.14" y2="147.32" width="0.1524" layer="91"/>
-<pinref part="IC2" gate="G$1" pin="9"/>
+<pinref part="MPU-6050" gate="G$1" pin="9"/>
 <pinref part="GND32" gate="1" pin="GND"/>
 </segment>
@@
 <junction x="805.18" y="134.62"/>
 <junction x="784.86" y="134.62"/>
-<pinref part="IC2" gate="G$1" pin="8"/>
+<pinref part="MPU-6050" gate="G$1" pin="8"/>
 <pinref part="C17" gate="G$1" pin="2"/>
 <pinref part="C20" gate="G$1" pin="1"/>
-<pinref part="IC2" gate="G$1" pin="13"/>
+<pinref part="MPU-6050" gate="G$1" pin="13"/>
 <pinref part="+3V8" gate="G$1" pin="+3V3"/>
 </segment>
@@
 <wire x1="896.62" y1="137.16" x2="896.62" y2="139.7" width="0.1524" layer="91"/>
 <wire x1="896.62" y1="139.7" x2="909.32" y2="139.7" width="0.1524" layer="91"/>
-<pinref part="IC2" gate="G$1" pin="24"/>
+<pinref part="MPU-6050" gate="G$1" pin="24"/>
 <label x="889" y="137.16" size="1.778" layer="95"/>
 </segment>
@@
 <segment>
 <wire x1="863.6" y1="142.24" x2="909.32" y2="142.24" width="0.1524" layer="91"/>
-<pinref part="IC2" gate="G$1" pin="23"/>
+<pinref part="MPU-6050" gate="G$1" pin="23"/>
 <label x="889" y="142.24" size="1.778" layer="95"/>
 </segment>
@@
 <net name="N$18" class="0">
 <segment>
-<pinref part="IC2" gate="G$1" pin="10"/>
+<pinref part="MPU-6050" gate="G$1" pin="10"/>
 <pinref part="C16" gate="G$1" pin="2"/>
 </segment>
@@
 <net name="N$19" class="0">
 <segment>
-<pinref part="IC2" gate="G$1" pin="20"/>
+<pinref part="MPU-6050" gate="G$1" pin="20"/>
 <pinref part="C21" gate="G$1" pin="1"/>
 <wire x1="805.18" y1="142.24" x2="802.64" y2="142.24" width="0.1524" layer="91"/>
