File: octanis_main_pcb_v0.3/octanis_v0.1.sch (EAGLE design)
At the start: 89 parts, among them IC1 REG1117, IC2 LM555D, Q1 32.768kHz, T1 BC547, T2 BC547, U1 BQ24210, U2 BQ27510_DRZ_12, U3 DRV8836DSSR, U4 DRV8836DSSR, U5 DRV8836DSSR, U6 MSP430F5529IPNR, U7 DRV8836DSSR, U9 BMP180

Commit message: startet new mainboard PCB
Parts:
- removed BATTERY: - BAT +, pinhead:PINHD-1X2
- removed C1, C2: 1uF, rcl:C-EUC1206
- removed C26: 12p, rcl:C-EUC0603
- removed C29: 100n, rcl:C-EUC0603
- removed C7, C8: 1uF, rcl:C-EUC0603
- removed CG1, CG3, CG6, CG7, CG8: 0.1uF, rcl:C-EUC0603
- removed CG2: 33nF, rcl:C-EUC0603
- removed CG4: 0.47uF, rcl:C-EUC0603
- removed DIGITAL1: DIGITAL1, pinhead:PINHD-1X6
- removed HEATPAD: HEATPAD, con-molex:22-23-2021
- removed HUMIDITY: HS1101, rcl:C-EU025-024X044
- removed I2C: SCL SDA, pinhead:PINHD-1X2
- removed IC1: REG1117, burr-brown:REG1117
- removed IC2: LM555D, linear:LM555D
- removed LED2: (no value), led:LEDCHIP-LED0603
- removed LED3: 5V-ok, adafruit:LEDCHIPLED_0603
- removed Q1: 32.768kHz, crystal:FC-12M
- removed R28: 0R, rcl:R-EU_R0603
- removed RG1: 1.8M, rcl:R-EU_R0603
- removed RG2: 18.2k, rcl:R-EU_R0603
- removed RG3, RH3: 1k, rcl:R-EU_R0603
- removed RG5, RG6: 100, rcl:R-EU_R0603
- removed RH1: 909k, rcl:R-EU_R0603
- removed RH2: 576k, rcl:R-EU_R0603
- removed RH4: 49.9k, rcl:R-EU_R0603
- removed RSBAT: 0.01, resistor:R-EU_R1206
- removed RT1: 21.5k, resistor:R-EU_R1206
- removed RVDM: float, resistor:R-EU_R1206
- removed SOLAR: - SOLAR +, pinhead:PINHD-1X2
- removed T1, T2: BC547, transistor:BC547
- removed TEMP1, TEMP2: 103AT, varistor:THERMISTOR-2,5
- removed U2: BQ27510_DRZ_12, bq27510_drz_12:BQ27510_DRZ_12
- removed U6: MSP430F5529IPNR, TI_MSP430_v16_intern:F552X---PN80
- added C22, C9: 12p, rcl:C-EUC0402
- added C23: 100n, rcl:C-EUC0402
- added C24: 100n, rcl:C-EUC0603
- added D5: 1N581D1206, lpatiny:1N581D1206
- added GREEN: 3V-ok, adafruit:LEDCHIPLED_0603
- added JP3: (no value), pinhead:PINHD-1X6
- added JP4: (no value), pinhead:PINHD-2X7
- added LED0: LED0, adafruit:LEDCHIPLED_0603
- added Q2: 32.768kHz, microcrystal:MS3V-T1R
- added R17, R8, R9: 1k, rcl:R-EU_R0603
- added R18, RPUC1, RPUD1: 10k, rcl:R-EU_R0603
- added R7: 0R, rcl:R-EU_R0402
- added RED: 5V-ok, adafruit:LEDCHIPLED_0603
- added U$2: F54XX[A]---PZ100, TI_MSP430_v16:F54XX[A]---PZ100
- added U$3: SST25VF064C, BertaLib:SST25VF064C
- added U$4: HX1, Octanis1:HX1
- ANALOG: device pinhead:PINHD-1X6 -> pinhead:PINHD-1X8
- C25: value 12p -> 100n
- DIGITAL2: device pinhead:PINHD-1X8 -> pinhead:PINHD-1X11
- JP1: value rst SBW tst -> RST TST
- JP2: value SERIAL -> (none); device pinhead:PINHD-1X4 -> pinhead:PINHD-1X2
- LED1: value (none) -> LED1; device led:LEDCHIP-LED0603 -> adafruit:LEDCHIPLED_0603
- R1: value 1k -> 10k
- R16: value 1M -> 10k
- R2: value 1k -> 1M
- R4: value 500 -> 1k; device resistor:R-EU_R1206 -> rcl:R-EU_R0603
- U1: value BQ24210 -> SHT21; device bq24210_dqc_10:BQ24210_DQC_10 -> SENSIRION-SHT21:SHT21
Connections:
- removed net AVCC: C29.1, R28.1, U6.11
- removed net BAT+: BATTERY.1, C2.1, C3.1, C7.1, CG3.1, IC1.VIN, L1.1, R1.2, R2.2, T2.C, U$1.VIN, U1.BAT, U2.BAT, U2.REGIN
- removed net BAT-: BATTERY.2, RG6.1, RSBAT.1
- removed net CHG_EN: U1.*EN, U6.5
- removed net EN_BAT_HEAT: T2.B
- removed net EN_SOLAR_HEAT: T1.B
- removed net HUMOUT: RH3.1
- removed net M1234SLEEP: U3.MODE, U3.NSLEEP, U4.MODE, U4.NSLEEP, U6.21
- removed net M5678SLEEP: U5.MODE, U5.NSLEEP, U6.35, U7.MODE, U7.NSLEEP
- removed net N$29: HUMIDITY.1, IC2.THR, IC2.TR, RH2.2
- removed net N$3: LED2.A, R2.1
- removed net N$33: RG2.1, RG3.2, TEMP2.1
- removed net N$34: CG1.1, RG3.1, U2.TS
- removed net N$35: CG4.1, RG1.2, U2.REG25, U2.VCC
- removed net N$36: CG6.1, CG7.1, RG5.2, U2.SRN
- removed net N$37: HEATPAD-1.S, T1.E, T2.E
- removed net N$38: CG6.2, CG8.2, RG6.2, U2.SRP
- removed net N$8: RT1.2, U1.VTSB
- removed net P2.7: DIGITAL1.6, U6.36
- removed net P3.0: DIGITAL1.5, U6.37
- removed net P3.1: DIGITAL1.4, U6.38
- removed net P3.2: DIGITAL1.3, U6.39
- removed net P3.3: DIGITAL1.2, U6.40
- removed net P3.4: DIGITAL1.1, U6.41
- removed net P3.5: U6.42
- removed net P3.6: U6.43
- removed net P3.7: U6.44
- removed net P5.0: ANALOG.2, U6.9
- removed net P5.1: ANALOG.1, U6.10
- removed net P5.4/XIN: C26.2, Q1.2, U6.12
- removed net P5.5/XOUT: C25.2, Q1.1, U6.13
- removed net P6.0: U6.77
- removed net P6.1: U6.78
- removed net P6.2: U6.79
- removed net P6.3: U6.80
- removed net P6.4: ANALOG.6, U6.1
- removed net P6.5: ANALOG.5, U6.2
- removed net P6.6: ANALOG.4, U6.3
- removed net P6.7: ANALOG.3, U6.4
- removed net RST/SBWTDIO: JP1.1, U6.76
- removed net SPI_CLK: JP2.1, U6.45
- removed net TARGET_DP: U6.62
- removed net TARGET_PUR: R16.2, U6.63
- removed net TEST/SBWTCK: JP1.2, U6.71
- removed net VCC: C1.1, SOLAR.2, T1.C, U1.VBUS
- new net 3.3V: C3.1, GREEN.A, JP4.7, JP4.8, L1.1, R1.2, R16.2, R2.2, U$1.VIN, U$3.HOLD, U$3.VCC, U$3.WP
- new net AVCC1: C23.1, R7.1, U$2.11
- new net CS: R17.2
- new net FMOSI: D5.A, R1.1, U$3.MOSI
- new net HX1EN: U$4.EN
- new net HX1TX: U$4.TXD
- new net LED0: LED0.A, U$2.9
- new net LED1: LED1.A, U$2.10
- new net M12SLEEP: U$2.18, U3.MODE, U3.NSLEEP
- new net M34SLEEP: U$2.23, U4.MODE, U4.NSLEEP
- new net M56SLEEP: U$2.40
- new net M78SLEEP: U$2.45, U5.MODE, U5.NSLEEP, U7.MODE, U7.NSLEEP
- new net N$28: ANALOG.7, U$2.98
- new net N$73: ANALOG.5, U$2.100
- new net N$74: ANALOG.4, U$2.1
- new net N$75: ANALOG.3, U$2.2
- new net N$76: ANALOG.2, U$2.3
- new net N$77: ANALOG.1, U$2.4
- new net N$78: DIGITAL2.10, U$2.77
- new net N$79: DIGITAL2.11, U$2.76
- new net P5.4/XIN1: C22.2, Q2.2, U$2.13
- new net P5.5/XOUT1: C9.2, Q2.1, U$2.14
- new net RST: JP1.1, U$2.96
- new net SCL2: JP4.2, RPUC.1, U$2.70
- new net SDA2: JP4.1, RPUD.1, U$2.69
- new net SPI_MISO: U$3.MISO
- new net SPI_SCK: JP3.3, R18.1, U$2.68
- new net SPI_SIMO: D5.C, JP3.5, U$2.72
- new net SPI_SOMI: JP3.6, U$2.73
- new net TST: JP1.2, U$2.91
- net +3V3: now also C24.1, C25.1, R7.2, RPUC1.2, RPUD1.2, U$2.16, U$2.38, U$2.64, U$2.87; no longer C8.1, IC1.VOUT, IC2.R, IC2.V+, R28.2, RH4.1, U6.18, U6.50
- net +5V: now also JP4.13, JP4.14, RED.A; no longer LED3.A
- net 5VEN: now also R2.1; no longer U6.6
- net GND: now also C22.1, C23.2, C24.2, C25.2, C9.1, JP4.11, JP4.12, JP4.3, JP4.4, JP4.5, JP4.6, Q2.GND, R8.1, R9.1, U$2.12, U$2.15, U$2.37, U$2.63, U$2.88, U$3.GND; no longer C1.2, C2.2, C25.1, C26.1, C29.2, C7.2, C8.2, CG1.2, CG2.2, CG3.2, CG4.2, CG7.2, CG8.1, HEATPAD-2.S, HUMIDITY.2, IC1.GND, IC2.GND, R16.1, RG5.1, RH1.1, RSBAT.2, RVDM.1, SOLAR.1, TEMP1.1, TEMP2.2, U1.EPAD, U2.EPAD, U2.EPAD1, U2.EPAD2, U2.EPAD3, U2.EPAD4, U2.EPAD5, U2.EPAD6, U2.VSS, U6.14, U6.19, U6.49, U6.61, U6.68
- net M1IN1: now also U$2.19; no longer U6.15
- net M1IN2: now also U$2.20; no longer U6.22
- net M2IN1: now also U$2.21; no longer U6.16
- net M2IN2: now also U$2.22; no longer U6.23
- net M3IN1: now also U$2.24; no longer U6.17
- net M3IN2: now also U$2.26; no longer U6.24
- net M4IN1: now also U$2.27; no longer U6.25
- net M4IN2: now also U$2.28; no longer U6.26
- net M5IN1: now also U$2.41; no longer U6.27
- net M5IN2: now also U$2.42; no longer U6.28
- net M6IN1: now also U$2.43; no longer U6.29
- net M6IN2: now also U$2.44; no longer U6.30
- net M7IN1: now also U$2.46; no longer U6.31
- net M7IN2: now also U$2.47; no longer U6.32
- net M8IN1: now also U$2.48; no longer U6.33
- net M8IN2: now also U$2.49; no longer U6.34
- net N$1: now also R18.2, U$3.SCK; no longer CG2.1, RG1.1, RG2.2, U2.BI/TOUT
- net N$10: now also R16.1, R17.1, U$3.CS; no longer R4.2, U1.ISET
- net N$14: now also U$2.86; no longer U6.60
- net N$15: now also U$2.85; no longer U6.59
- net N$2: now also U1.VDD; no longer LED1.A, R1.1
- net N$20: now also U$2.84; no longer U6.58
- net N$21: now also U$2.83; no longer U6.57
- net N$22: now also U$2.82; no longer U6.56
- net N$23: now also U$2.81; no longer U6.55
- net N$24: now also U$2.80; no longer U6.54
- net N$26: now also U$2.79; no longer U6.53
- net N$27: now also ANALOG.8, U$2.97; no longer IC2.CV, RH1.2
- net N$30: now also ANALOG.6, U$2.99; no longer IC2.DIS, RH2.1, RH4.2
- net N$31: now also DIGITAL2.9, U$2.78; no longer IC2.Q, RH3.2
- net N$4: now also GREEN.C, R4.2; no longer LED1.C, U1.*CHG
- net N$44: now also RED.C; no longer LED3.C
- net N$5: now also LED0.C, R8.2; no longer LED2.C, U1.*PG
- net N$6: now also LED1.C, R9.2; no longer RVDM.2, U1.VDPM
- net N$7: now also JP4.10, JP4.9; no longer RT1.1, TEMP1.2, U1.TS
- net RX: now also JP2.1, U$2.54; no longer JP2.3, U6.52
- net SCL: now also JP3.1, RPUC1.1, U$2.35, U1.SCL; no longer I2C.1, RPUC.1, U2.SCL, U6.47
- net SDA: now also JP3.2, RPUD1.1, U$2.34, U1.SDA; no longer I2C.2, RPUD.1, U2.SDA, U6.46
- net SPI_SLAVE_EN: now also JP3.4, U$2.71; no longer JP2.4, U6.48
- net TX: now also U$2.53; no longer U6.51
- net VCORE: now also U$2.62; no longer U6.20
Other:
- note added: "Flash Memory"
- note added: "Gyroscope/Accelerometer"
- note added: "I2C Pull-up Resistor for EPS"
- note added: "Sensirion Humidity Sensor"
- note removed: "Battery Charging"
- note removed: "Fuel Gauge"
- note removed: "Main MSP430F5529 w Power, Clock and USB"
- note removed: "On-Board Heating"
- moved on the sheet: C14, C16, C17, C18, C19, C20, C21, C25, C3, C30, C4, C5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

Commit message: added aria bob
Parts:
- removed RPUC1, RPUD1: 10k, rcl:R-EU_R0603
- added RPUC2, RPUD2: 10k, rcl:R-EU_R0603
Connections:
- net +3V3: now also RPUC2.2, RPUD2.2; no longer RPUC1.2, RPUD1.2
- net SCL: now also RPUC.1; no longer RPUC1.1
- net SCL2: now also RPUC2.1; no longer RPUC.1
- net SDA: now also RPUD.1; no longer RPUD1.1
- net SDA2: now also RPUD2.1; no longer RPUD.1
Other:
- moved on the sheet: RPUC, RPUD
Changed lines of the file:
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@@
 <part name="GND67" library="supply1" deviceset="GND" device=""/>
 <part name="+3V3" library="supply1" deviceset="+3V3" device=""/>
-<part name="RPUD" library="rcl" deviceset="R-EU_" device="R0603" value="10k"/>
-<part name="RPUC" library="rcl" deviceset="R-EU_" device="R0603" value="10k"/>
+<part name="RPUD2" library="rcl" deviceset="R-EU_" device="R0603" value="10k"/>
+<part name="RPUC2" library="rcl" deviceset="R-EU_" device="R0603" value="10k"/>
 <part name="+3V6" library="supply1" deviceset="+3V3" device=""/>
 <part name="U$1" library="texas" deviceset="TPS61230" device=""/>
@@
 <part name="Q2" library="microcrystal" deviceset="MS3V-T1R" device="" value="32.768kHz"/>
 <part name="JP2" library="pinhead" deviceset="PINHD-1X2" device=""/>
-<part name="RPUD1" library="rcl" deviceset="R-EU_" device="R0603" value="10k"/>
-<part name="RPUC1" library="rcl" deviceset="R-EU_" device="R0603" value="10k"/>
+<part name="RPUD" library="rcl" deviceset="R-EU_" device="R0603" value="10k"/>
+<part name="RPUC" library="rcl" deviceset="R-EU_" device="R0603" value="10k"/>
 <part name="+3V1" library="supply1" deviceset="+3V3" device=""/>
 <part name="JP3" library="pinhead" deviceset="PINHD-1X6" device=""/>
@@
 <attribute name="VALUE" x="436.88" y="266.7" size="1.778" layer="96"/>
 </instance>
-<instance part="RPUD" gate="G$1" x="558.8" y="312.42" rot="R90"/>
-<instance part="RPUC" gate="G$1" x="566.42" y="312.42" rot="R90"/>
+<instance part="RPUD2" gate="G$1" x="558.8" y="312.42" rot="R90"/>
+<instance part="RPUC2" gate="G$1" x="566.42" y="312.42" rot="R90"/>
 <instance part="+3V6" gate="G$1" x="558.8" y="327.66" smashed="yes">
 <attribute name="VALUE" x="558.8" y="327.66" size="1.778" layer="96"/>
@@
 </instance>
 <instance part="JP2" gate="G$1" x="426.72" y="231.14"/>
-<instance part="RPUD1" gate="G$1" x="520.7" y="312.42" rot="R90"/>
-<instance part="RPUC1" gate="G$1" x="528.32" y="312.42" rot="R90"/>
+<instance part="RPUD" gate="G$1" x="520.7" y="312.42" rot="R90"/>
+<instance part="RPUC" gate="G$1" x="528.32" y="312.42" rot="R90"/>
 <instance part="+3V1" gate="G$1" x="520.7" y="327.66" smashed="yes">
 <attribute name="VALUE" x="520.7" y="327.66" size="1.778" layer="96"/>
@@
 <segment>
 <pinref part="+3V6" gate="G$1" pin="+3V3"/>
-<pinref part="RPUD" gate="G$1" pin="2"/>
+<pinref part="RPUD2" gate="G$1" pin="2"/>
 <wire x1="558.8" y1="325.12" x2="558.8" y2="320.04" width="0.1524" layer="91"/>
-<pinref part="RPUC" gate="G$1" pin="2"/>
+<pinref part="RPUC2" gate="G$1" pin="2"/>
 <wire x1="558.8" y1="320.04" x2="558.8" y2="317.5" width="0.1524" layer="91"/>
 <wire x1="558.8" y1="320.04" x2="566.42" y2="320.04" width="0.1524" layer="91"/>
@@
 <segment>
 <pinref part="+3V1" gate="G$1" pin="+3V3"/>
-<pinref part="RPUD1" gate="G$1" pin="2"/>
+<pinref part="RPUD" gate="G$1" pin="2"/>
 <wire x1="520.7" y1="325.12" x2="520.7" y2="320.04" width="0.1524" layer="91"/>
-<pinref part="RPUC1" gate="G$1" pin="2"/>
+<pinref part="RPUC" gate="G$1" pin="2"/>
 <wire x1="520.7" y1="320.04" x2="520.7" y2="317.5" width="0.1524" layer="91"/>
 <wire x1="520.7" y1="320.04" x2="528.32" y2="320.04" width="0.1524" layer="91"/>
@@
 </segment>
 <segment>
-<pinref part="RPUD1" gate="G$1" pin="1"/>
+<pinref part="RPUD" gate="G$1" pin="1"/>
 <wire x1="520.7" y1="307.34" x2="525.78" y2="307.34" width="0.1524" layer="91"/>
 <label x="525.78" y="289.56" size="1.778" layer="95" rot="R90"/>
@@
 </segment>
 <segment>
-<pinref part="RPUC1" gate="G$1" pin="1"/>
+<pinref part="RPUC" gate="G$1" pin="1"/>
 <label x="528.32" y="289.56" size="1.778" layer="95" rot="R90"/>
 <wire x1="528.32" y1="307.34" x2="528.32" y2="274.32" width="0.1524" layer="91"/>
@@
 <label x="558.8" y="297.18" size="1.778" layer="95" rot="R90"/>
 <wire x1="558.8" y1="307.34" x2="558.8" y2="294.64" width="0.1524" layer="91"/>
-<pinref part="RPUD" gate="G$1" pin="1"/>
+<pinref part="RPUD2" gate="G$1" pin="1"/>
 <wire x1="558.8" y1="304.8" x2="558.8" y2="307.34" width="0.1524" layer="91"/>
 </segment>
@@
 </segment>
 <segment>
-<pinref part="RPUC" gate="G$1" pin="1"/>
+<pinref part="RPUC2" gate="G$1" pin="1"/>
 <label x="566.42" y="297.18" size="1.778" layer="95" rot="R90"/>
 <wire x1="566.42" y1="307.34" x2="566.42" y2="294.64" width="0.1524" layer="91"/>

Commit message: starting layout v0.3
Parts:
- removed R5: 68k, rcl:R-EU_R0603
- removed RPUC2, RPUD2: 10k, rcl:R-EU_R0603
- added C1: 100n, rcl:C-EUC0603
- added C2: 100nF, rcl:C-EUC0603
- added C26, C27, C28, C8: 470n, rcl:C-EUC0603
- added C7: 22uF, rcl:C-EUC0603
- added SJ1: (no value), jumper:SJ2W
- C15: value 0.1uF -> 100nF
- R3: value 270k -> 1M
- U$1: value TPS61230 -> TPS61232; device texas:TPS61230 -> texasinstruments:TPS61232
Connections:
- net SPI_SLAVE_EN renamed SPI_EXTSLAVE_TE
- removed net CS: R17.2
- removed net HX1TX: U$4.TXD
- removed net M12SLEEP: U$2.18, U3.MODE, U3.NSLEEP
- removed net M34SLEEP: U$2.23, U4.MODE, U4.NSLEEP
- removed net M56SLEEP: U$2.40
- removed net M78SLEEP: U$2.45, U5.MODE, U5.NSLEEP, U7.MODE, U7.NSLEEP
- removed net N$43: R3.1, R5.2, U$1.FB
- removed net N$7: JP4.10, JP4.9
- new net M1234SLEEP: U$2.24, U3.MODE, U3.NSLEEP, U4.MODE, U4.NSLEEP
- new net M5678SLEEP: U$2.50, U5.MODE, U5.NSLEEP, U7.MODE, U7.NSLEEP
- new net RFGND: U$4.RFGND, U$4.RFGND2
- new net SPI_FLASH_CS: R17.2, U$2.75
- new net V_MOTOR: C26.2, C27.2, C28.2, C8.2, SJ1.2, U3.VCC, U4.VCC, U5.VCC, U7.VCC
- net +3V3: now also C1.1, C3.1, GREEN.A, JP4.10, JP4.7, JP4.8, JP4.9, L1.1, R1.2, R16.2, R2.2, SJ1.1, U$1.VIN, U$3.HOLD, U$3.VCC, U1.VDD; no longer RPUC2.2, RPUD2.2
- net +5V: now also C2.1, C7.1, SJ1.3, U$1.FB, U$4.VCC; no longer U3.VCC, U4.VCC, U5.VCC, U7.VCC
- net 3.3V: no longer C3.1, GREEN.A, JP4.7, JP4.8, L1.1, R1.2, R16.2, R2.2, U$1.VIN, U$3.HOLD, U$3.VCC
- net 5VEN: now also U$2.17
- net GND: now also C1.2, C2.2, C26.1, C27.1, C28.1, C7.2, C8.1, U$4.0V; no longer R5.1
- net M1IN1: now also U$2.25; no longer U$2.19
- net M1IN2: now also U$2.26; no longer U$2.20
- net M2IN1: now also U$2.27; no longer U$2.21
- net M2IN2: now also U$2.28; no longer U$2.22
- net M3IN1: now also U$2.42; no longer U$2.24
- net M3IN2: now also U$2.43; no longer U$2.26
- net M4IN1: now also U$2.44; no longer U$2.27
- net M4IN2: now also U$2.45; no longer U$2.28
- net M5IN1: now also U$2.46; no longer U$2.41
- net M5IN2: now also U$2.47; no longer U$2.42
- net M6IN1: now also U$2.48; no longer U$2.43
- net M6IN2: now also U$2.49; no longer U$2.44
- net M7IN1: now also U$2.56; no longer U$2.46
- net M7IN2: now also U$2.57; no longer U$2.47
- net M8IN1: now also U$2.58; no longer U$2.48
- net M8IN2: now also U$2.59; no longer U$2.49
- net N$2: now also R3.1, U$1.PG; no longer U1.VDD
- net SCL: now also JP4.2
- net SCL2: no longer JP4.2, RPUC2.1
- net SDA: now also JP4.1
- net SDA2: no longer JP4.1, RPUD2.1
- net TX: now also U$4.TXD
Other:
- note removed: "I2C Pull-up Resistor for EPS"

Commit message: layout done
Parts:
- removed D5: 1N581D1206, lpatiny:1N581D1206
- removed R1, R18: 10k, rcl:R-EU_R0603
- removed R17: 1k, rcl:R-EU_R0603
- added SJ2: (no value), jumper:SJ
- C10: value 4.7uF -> 4.7u
- C11: value 0.1uF -> 100n
- C12: value 10uF -> 10u
- C13: value 0.22uF -> 220n
- C15, C16, C2, C20: value 100nF -> 100n
- C17: value 10nF -> 10n
- C21: value 2,2nF -> 2.2n
- C7: value 22uF -> 3 x 22uF
- DIGITAL2: value DIGITAL2 -> DIGITAL I/O
- JP2: value (none) -> TX RX
- JP3: value (none) -> SPI; device pinhead:PINHD-1X6 -> pinhead:PINHD-1X4
- U$2: value F54XX[A]---PZ100 -> MSP430F5438A
Connections:
- removed net FMOSI: D5.A, R1.1, U$3.MOSI
- removed net N$1: R18.2, U$3.SCK
- removed net N$10: R16.1, R17.1, U$3.CS
- removed net SPI_SIMO: D5.C, JP3.5, U$2.72
- removed net SPI_SOMI: JP3.6, U$2.73
- new net SPI_MOSI: JP3.3, U$2.72, U$3.MOSI
- net +3V3: no longer R1.2
- net 5VEN: now also U$2.23; no longer U$2.17
- net GND: now also SJ2.1
- net HX1EN: now also U$2.52
- net RFGND: now also SJ2.2
- net SCL: now also RPUD.1; no longer JP3.1, RPUC.1
- net SDA: now also RPUC.1; no longer JP3.2, RPUD.1
- net SPI_EXTSLAVE_TE: now also JP3.2; no longer JP3.4
- net SPI_FLASH_CS: now also R16.1, U$3.CS; no longer R17.2
- net SPI_MISO: now also JP3.4, U$2.73
- net SPI_SCK: now also JP3.1, U$3.SCK; no longer JP3.3, R18.1
Other:
- moved on the sheet: C4, RPUC, RPUD

Commit message: replaced sensirion humidity sensor with bosch
Parts:
- removed C1, C11: 100n, rcl:C-EUC0603
- removed C12: 10u, resistor:CPOL-EUA/3216-18R
- removed U1: SHT21, SENSIRION-SHT21:SHT21
- removed U9: BMP180, SparkFun-Sensors:BMP180
- added C29: 100n, rcl:C-EUC0603
- added IC1: BME280, bosch-bme280:BME280
- added JP5: (no value), pinhead:PINHD-2X2
- ANALOG: value ANALOG -> A7:A0
Connections:
- net +3V3: now also C29.1, IC1.CSB, IC1.VDD, IC1.VDDIO, JP5.1; no longer C1.1, C11.1, C12.+, U1.VDD, U9.VDD, U9.VDDIO
- net GND: now also C29.2, IC1.GND, IC1.SDO, JP5.2; no longer C1.2, C11.2, C12.-, U1.VSS, U9.GND
- net SCL: now also IC1.SCK, JP5.4; no longer U1.SCL, U9.SCL
- net SDA: now also IC1.SDI, JP5.3; no longer U1.SDA, U9.SDA
Other:
- note added: "Bosch Pressure/Humidity"
- note removed: "Pressure Sensor"
- note removed: "Sensirion Humidity Sensor"
