File: octanis_main_pcb_v0.3/octanis_v0.1.brd (EAGLE design)
At the start: 75.6 x 41.9 mm, 67 parts, among them IC1 BME280, Q2 32.768kHz, U3 DRV8836DSSR, U4 DRV8836DSSR, U5 DRV8836DSSR, U7 DRV8836DSSR

Commit message: added holes
Routing:
- net N$78: track 27.1 -> 30.0 mm
- net HX1EN: track 24.5 -> 27.3 mm
- net RFGND: track 105.4 -> 107.6 mm
Changed lines of the file:
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@@
 <layer number="43" name="vRestrict" color="2" fill="10" visible="no" active="yes"/>
 <layer number="44" name="Drills" color="7" fill="1" visible="no" active="yes"/>
-<layer number="45" name="Holes" color="7" fill="1" visible="no" active="yes"/>
+<layer number="45" name="Holes" color="7" fill="1" visible="yes" active="yes"/>
 <layer number="46" name="Milling" color="3" fill="1" visible="no" active="yes"/>
 <layer number="47" name="Measures" color="7" fill="1" visible="no" active="yes"/>
@@
 <rectangle x1="21.9583" y1="34.5313" x2="23.1775" y2="34.5567" layer="200"/>
 <rectangle x1="22.1615" y1="34.5567" x2="22.9997" y2="34.5821" layer="200"/>
+<hole x="12.7" y="34.29" drill="3"/>
+<hole x="60.96" y="34.29" drill="3"/>
+<hole x="60.96" y="7.62" drill="3"/>
 </plain>
 <attributes>
@@
 <polygon width="0.3048" layer="1" spacing="0.0254" thermals="no">
 <vertex x="23.3172" y="5.3721"/>
-<vertex x="58.8899" y="5.3975"/>
-<vertex x="58.9153" y="6.0325"/>
+<vertex x="58.2803" y="5.3975"/>
+<vertex x="58.3057" y="6.0325"/>
 <vertex x="23.3172" y="6.0071"/>
 </polygon>
@@
 <wire x1="64.4652" y1="3.556" x2="65.6844" y2="3.4036" width="0.6096" layer="16"/>
 <wire x1="65.6844" y1="3.4036" x2="65.1256" y2="3.5052" width="0.6096" layer="16"/>
-<via x="58.4073" y="5.7658" extent="1-16" drill="0.3"/>
+<via x="57.7977" y="5.7658" extent="1-16" drill="0.3"/>
 <wire x1="26.3008" y1="11.4808" x2="27.9942" y2="11.4808" width="0.254" layer="1"/>
 <wire x1="27.9942" y1="11.4808" x2="28.194" y2="11.6806" width="0.254" layer="1"/>
@@
 <wire x1="11.6638" y1="25.329" x2="10.8712" y2="24.5364" width="0.3048" layer="1"/>
 <wire x1="10.8712" y1="24.5364" x2="10.8712" y2="24.0284" width="0.3048" layer="1"/>
+<wire x1="57.7977" y1="5.7658" x2="63.0682" y2="4.2164" width="0" layer="19" extent="1-1"/>
 </signal>
 <signal name="N$9">
@@
 <wire x1="41.394" y1="24.13" x2="37.9476" y2="24.13" width="0.3048" layer="1"/>
 <wire x1="61.6458" y1="18.3896" x2="62.9158" y2="18.3896" width="0.3048" layer="1"/>
-<wire x1="63.9064" y1="30.5308" x2="52.4764" y2="30.5308" width="0.3048" layer="1"/>
-<wire x1="52.4764" y1="30.5308" x2="52.4764" y2="26.2636" width="0.3048" layer="1"/>
+<wire x1="63.9064" y1="30.3784" x2="52.4764" y2="30.3784" width="0.3048" layer="1"/>
+<wire x1="52.4764" y1="30.3784" x2="52.4764" y2="26.2636" width="0.3048" layer="1"/>
 <wire x1="52.4764" y1="26.2636" x2="47.8028" y2="26.2636" width="0.3048" layer="1"/>
 <wire x1="47.8028" y1="26.2636" x2="46.7868" y2="25.2476" width="0.3048" layer="1"/>
 <wire x1="46.7868" y1="25.2476" x2="41.5464" y2="25.2476" width="0.3048" layer="1"/>
 <wire x1="41.5464" y1="25.2476" x2="41.394" y2="25.4" width="0.3048" layer="1"/>
-<wire x1="63.9064" y1="30.5308" x2="63.9064" y2="29.464" width="0.3048" layer="1"/>
+<wire x1="63.9064" y1="30.3784" x2="63.9064" y2="29.464" width="0.3048" layer="1"/>
 <wire x1="63.9064" y1="29.464" x2="63.9064" y2="18.3896" width="0.3048" layer="1"/>
 <wire x1="63.9064" y1="18.3896" x2="62.9158" y2="18.3896" width="0.3048" layer="1"/>
@@
 <contactref element="DIGITAL2" pad="9"/>
 <wire x1="45.894" y1="27.1294" x2="45.894" y2="32.8676" width="0.254" layer="1"/>
-<wire x1="45.894" y1="32.8676" x2="58.9788" y2="32.8676" width="0.254" layer="1"/>
-<wire x1="58.9788" y1="32.8676" x2="58.9788" y2="39.116" width="0.254" layer="1"/>
+<wire x1="45.894" y1="32.8676" x2="58.5216" y2="32.8676" width="0.254" layer="1"/>
+<wire x1="58.5216" y1="32.8676" x2="58.5216" y2="39.0144" width="0.254" layer="1"/>
+<wire x1="58.5216" y1="39.0144" x2="58.9788" y2="39.0144" width="0.254" layer="1"/>
+<wire x1="58.9788" y1="39.0144" x2="58.9788" y2="39.116" width="0.254" layer="1"/>
 </signal>
 <signal name="N$78">
 <contactref element="U$2" pad="77"/>
 <contactref element="DIGITAL2" pad="10"/>
-<wire x1="46.394" y1="27.1294" x2="46.394" y2="32.1564" width="0.254" layer="1"/>
-<wire x1="46.394" y1="32.1564" x2="61.5188" y2="32.1564" width="0.254" layer="1"/>
-<wire x1="61.5188" y1="32.1564" x2="61.5188" y2="39.116" width="0.254" layer="1"/>
+<wire x1="46.394" y1="27.1294" x2="46.394" y2="31.5976" width="0.254" layer="1"/>
+<wire x1="46.394" y1="31.5976" x2="63.5" y2="31.5976" width="0.254" layer="1"/>
+<wire x1="63.5" y1="31.5976" x2="63.5" y2="36.6268" width="0.254" layer="1"/>
+<wire x1="63.5" y1="36.6268" x2="61.8744" y2="38.1" width="0.254" layer="1"/>
+<wire x1="61.8744" y1="38.1" x2="61.8744" y2="38.7604" width="0.254" layer="1"/>
+<wire x1="61.8744" y1="38.7604" x2="61.5188" y2="39.116" width="0.254" layer="1"/>
 </signal>
 <signal name="N$79">
 <contactref element="U$2" pad="76"/>
 <contactref element="DIGITAL2" pad="11"/>
-<wire x1="46.894" y1="27.1294" x2="46.894" y2="31.3944" width="0.254" layer="1"/>
-<wire x1="46.894" y1="31.3944" x2="64.0588" y2="31.3944" width="0.254" layer="1"/>
-<wire x1="64.0588" y1="31.3944" x2="64.0588" y2="39.116" width="0.254" layer="1"/>
+<wire x1="46.894" y1="27.1294" x2="46.894" y2="31.0388" width="0.254" layer="1"/>
+<wire x1="46.894" y1="31.0388" x2="64.0588" y2="31.0388" width="0.254" layer="1"/>
+<wire x1="64.0588" y1="31.0388" x2="64.0588" y2="39.116" width="0.254" layer="1"/>
 </signal>
 <signal name="SPI_SCK">
@@
 <wire x1="54.0004" y1="9.906" x2="54.2798" y2="10.1854" width="0.254" layer="1"/>
 <via x="54.2798" y="10.1854" extent="1-16" drill="0.3"/>
-<wire x1="54.2798" y1="10.1854" x2="58.3692" y2="10.1854" width="0.254" layer="16"/>
-<via x="58.3692" y="10.1854" extent="1-16" drill="0.3"/>
-<wire x1="58.3692" y1="10.1854" x2="60.452" y2="10.1854" width="0.254" layer="1"/>
-<wire x1="60.452" y1="10.1854" x2="65.151" y2="14.8844" width="0.254" layer="1"/>
-<wire x1="65.151" y1="14.8844" x2="67.818" y2="14.8844" width="0.254" layer="1"/>
+<wire x1="54.2798" y1="10.1854" x2="57.5564" y2="10.1854" width="0.254" layer="16"/>
+<via x="57.5564" y="10.1854" extent="1-16" drill="0.3"/>
+<wire x1="57.5564" y1="10.1854" x2="57.5564" y2="14.8844" width="0.254" layer="1"/>
+<wire x1="57.5564" y1="14.8844" x2="67.818" y2="14.8844" width="0.254" layer="1"/>
 <wire x1="67.818" y1="14.8844" x2="67.9704" y2="15.0368" width="0.254" layer="1"/>
 </signal>
@@
 <wire x1="37.3888" y1="7.874" x2="50.4952" y2="7.874" width="0.6096" layer="16"/>
 <wire x1="50.4952" y1="7.874" x2="51.2572" y2="7.112" width="0.6096" layer="16"/>
-<wire x1="51.2572" y1="7.112" x2="64.6176" y2="7.112" width="0.6096" layer="16"/>
-<wire x1="64.6176" y1="7.112" x2="65.278" y2="5.2324" width="0.6096" layer="16"/>
-<wire x1="65.278" y1="5.2324" x2="71.2216" y2="5.1816" width="0.6096" layer="16"/>
-<wire x1="71.2216" y1="5.1816" x2="71.2216" y2="32.8168" width="0.6096" layer="16"/>
+<wire x1="51.2572" y1="7.112" x2="58.2168" y2="7.112" width="0.6096" layer="16"/>
+<wire x1="58.2168" y1="7.112" x2="59.182" y2="4.0132" width="0.6096" layer="16"/>
+<wire x1="59.182" y1="4.0132" x2="71.2216" y2="3.9624" width="0.6096" layer="16"/>
+<wire x1="71.2216" y1="3.9624" x2="71.2216" y2="32.8168" width="0.6096" layer="16"/>
 <wire x1="71.2216" y1="32.8168" x2="71.2724" y2="37.2364" width="0.6096" layer="16"/>
 <wire x1="71.2724" y1="37.2364" x2="71.2724" y2="37.8968" width="0.6096" layer="16"/>
