File: octanis_main_pcb_v0.4/octanis_v0.4.brd (EAGLE design)
At the start: 76.2 x 41.9 mm, 69 parts, among them IC1 BME280, Q2 32.768kHz, U3 DRV8836DSSR, U4 DRV8836DSSR, U5 DRV8836DSSR, U7 DRV8836DSSR

Commit message: layout 0.4 almost done
Parts:
- removed SJ3: (no value), jumper:SJ
- added U$2: STARGND, lpatiny:STAR
- moved R9 50.4 mm to (65.2, 1.88), turned to 90 degrees
- moved R8 49.8 mm to (66.7, 1.91), turned to 90 degrees
- moved LED1 45.1 mm to (65.2, 5.87), turned to 180 degrees
- moved LED0 44.5 mm to (66.5, 5.84), turned to 180 degrees
- moved R16 12.4 mm to (12.4, 29.6), turned to 270 degrees
- moved JP1 4.09 mm to (26.2, 18.5), turned to 45 degrees
- moved JP3 1.60 mm to (19.2, 34.0)
- moved U$3 1.28 mm to (18.5, 28.6)
- moved C11 1.16 mm to (46.9, 33.2)
- moved C25 0.37 mm to (34.0, 16.9)
- moved C19 0.32 mm to (31.4, 12.0)
- moved C18 0.29 mm to (32.8, 15.7)
- moved C30 0.23 mm to (32.9, 13.1)
Connections:
- removed net P6.2/UCB1STE/C1.5: MSP1.76
- removed net P6.3/UCB1CLK/C1.4: MSP1.77
- removed net P6.4/UCB1SIMO/UCB1SDA/C1.3: MSP1.78
- removed net P6.5/UCB1SOMI/UCB1SCL/C1.2: MSP1.79
- removed net P6.6/TA2.3/UCB3SIMO/UCB3SDA/C1.1: MSP1.80
- net A14: now also MSP1.55; no longer MSP1.54
- net A15: now also MSP1.54; no longer MSP1.55
- net AGND: now also U$2.AGND; no longer SJ3.2
- net GND: now also U$2.DGND, U$2.GND; no longer SJ3.1
- net N$10: now also C9.2; no longer C22.2
- net N$8: now also C22.2; no longer C9.2
- net SPI_EXTSLAVE_TE: now also MSP1.76
- net SPI_FLASH_CS: now also MSP1.80
- net SPI_MISO: now also MSP1.79
- net SPI_MOSI: now also MSP1.78
- net SPI_SCK: now also MSP1.77
Routing:
- net +3V3: track 145.0 -> 212.5 mm, vias 4 -> 8
- net TX: track 0.00 -> 49.0 mm, vias 0 -> 2
- net SPI_FLASH_CS: track 0.00 -> 43.1 mm
- net AGND: track 26.0 -> 68.4 mm, vias 5 -> 7
- net SPI_MISO: track 0.00 -> 41.4 mm
- net SPI_MOSI: track 0.00 -> 36.5 mm
- net SPI_SCK: track 0.00 -> 34.1 mm
- net GND: track 57.3 -> 91.2 mm, vias 22 -> 25
- net SPI_EXTSLAVE_TE: track 0.00 -> 26.7 mm
- net M8IN2: track 0.00 -> 24.8 mm
- net SDA: track 44.6 -> 68.1 mm, vias 5 -> 8
- net SCL: track 38.6 -> 61.9 mm, vias 1 -> 4
- net N$14: track 0.00 -> 22.6 mm
- net N$38: track 0.00 -> 20.2 mm
- net N$15: track 0.00 -> 19.8 mm
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
Commit message: v0.4 layout finished
Parts:
- GPIO2: value DIGITAL I/O -> A18:A8
- R10: value 91 kW, 0.1%, ±25 ppm/°C -> 91k 0.1% ±25 ppm/°C
- SJ1: value (none) -> 3V3 V_Motor 5V
- moved R8 69.0 mm to (2.72, 27.7), turned to 0 degrees
- moved R9 68.2 mm to (2.69, 29.3), turned to 0 degrees
- moved LED0 63.8 mm to (6.65, 27.9), turned to 90 degrees
- moved C10 63.4 mm to (63.1, 8.31)
- moved C15 63.4 mm to (63.7, 0.69)
- moved COMPASS 63.4 mm to (63.8, 4.65)
- moved C13 63.4 mm to (66.0, 8.16)
- moved LED1 63.0 mm to (6.68, 29.3), turned to 90 degrees
- moved C2 1.27 mm to (29.5, 35.7)
- moved C19 0.83 mm to (30.9, 12.6)
- moved C11 0.29 mm to (46.7, 33.4)
- moved C30 0.07 mm to (32.9, 13.2)
- renumbered ANALOG to GPIO1, DIGITAL2 to GPIO2
Connections:
- net M12SLEEP renamed P2.0/PM_UCA1STE
- removed net HX1EN: U$4.EN
- removed net N$16: MSP1.18
- removed net N$29: MSP1.19
- removed net P5.6/TA2.1/VREF+/VEREF+/C1.7: MSP1.70
- removed net P5.7/TA2.2/VREF-/VEREF-/C1.6: MSP1.71
- removed net P9.3/TA3.4: MSP1.75
- new net HX1_EN: MSP1.70, U$4.EN
- net 5VEN: now also MSP1.17
- net LED0: now also MSP1.75
- net LED1: now also MSP1.71
- net M1234SLEEP: now also MSP1.18
- net M1IN1: now also MSP1.19; no longer MSP1.17
Routing:
- net +3V3: track 212.5 -> 268.7 mm, vias 8 -> 12
- net LED1: track 0.00 -> 53.3 mm, vias 0 -> 4
- net LED0: track 0.00 -> 53.1 mm, vias 0 -> 4
- net HX1_EN: track 0.00 -> 31.5 mm, vias 0 -> 4
- net 5VEN: track 6.49 -> 36.9 mm, vias 2 -> 4
- net GND: track 91.2 -> 120.1 mm, vias 25 -> 31
- net SCL: track 61.9 -> 86.5 mm, vias 4 -> 6
- net SDA: track 68.1 -> 92.3 mm, vias 8 -> 10
- net N$58: track 15.5 -> 0.00 mm
- net N$16: track 0.00 -> 13.1 mm
- net M1234SLEEP: track 17.7 -> 28.6 mm
- net +5V: track 101.7 -> 110.3 mm, vias 2 -> 3
- net N$1: track 3.34 -> 7.68 mm
- net N$62: track 3.32 -> 0.00 mm
- net RFGND: track 10.4 -> 12.9 mm
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Other:
- board size 76.2 x 41.9 mm -> 69.2 x 41.9 mm
- board text added: "3V3 V_mot 5V"
- board text added: "MISO MOSI TE CLK"
