File: octanis_main_pcb_v0.4/octanis_v0.4.sch (EAGLE design)
At the start: 69 parts, among them IC1 BME280, Q2 32.768kHz, U3 DRV8836DSSR, U4 DRV8836DSSR, U5 DRV8836DSSR, U7 DRV8836DSSR

Commit message: layout 0.4 almost done
Parts:
- removed SJ3: (no value), jumper:SJ
- added U$2: STARGND, lpatiny:STARGND
Connections:
- net A14: now also MSP1.P6.1/A14; no longer MSP1.P6.0/A15
- net A15: now also MSP1.P6.0/A15; no longer MSP1.P6.1/A14
- net AGND: now also U$2.AGND; no longer SJ3.2
- net GND: now also U$2.DGND, U$2.GND; no longer SJ3.1
- net N$10: now also C9.2; no longer C22.2
- net N$8: now also C22.2; no longer C9.2
- net SPI_EXTSLAVE_TE: now also MSP1.P6.2/UCB1STE/C1.5
- net SPI_FLASH_CS: now also MSP1.P6.6/TA2.3/UCB3SIMO/UCB3SDA/C1.1
- net SPI_MISO: now also MSP1.P6.5/UCB1SOMI/UCB1SCL/C1.2
- net SPI_MOSI: now also MSP1.P6.4/UCB1SIMO/UCB1SDA/C1.3
- net SPI_SCK: now also MSP1.P6.3/UCB1CLK/C1.4
Other:
- moved on the sheet: C22, C9

Commit message: v0.4 layout finished
Parts:
- GPIO2: value DIGITAL I/O -> A18:A8
- R10: value 91 kW, 0.1%, ±25 ppm/°C -> 91k 0.1% ±25 ppm/°C
- SJ1: value (none) -> 3V3 V_Motor 5V
- renumbered ANALOG to GPIO1, DIGITAL2 to GPIO2
Connections:
- removed net HX1EN: U$4.EN
- removed net M12SLEEP: MSP1.P2.0/PM_UCA1STE
- removed net N$16: MSP1.P2.2/PM_UCA1RXD/PM_UCA1SOMI
- removed net N$29: MSP1.P2.3/PM_UCA1TXD/PM_UCA1SIMO
- new net HX1_EN: MSP1.P5.6/TA2.1/VREF+/VEREF+/C1.7, U$4.EN
- net 5VEN: now also MSP1.P2.1/PM_UCA1CLK
- net LED0: now also MSP1.P9.3/TA3.4
- net LED1: now also MSP1.P5.7/TA2.2/VREF-/VEREF-/C1.6
- net M1234SLEEP: now also MSP1.P2.2/PM_UCA1RXD/PM_UCA1SOMI
- net M1IN1: now also MSP1.P2.3/PM_UCA1TXD/PM_UCA1SIMO; no longer MSP1.P2.1/PM_UCA1CLK
