File: pannelized v0_5/pannelized_v0_5.brd (EAGLE design)
At the start: 80 x 48 mm, 103 parts, among them IC1 BME280, IC2 BNO055A, Q1 32.768kHz, Q2 32.768kHz, U1 TPS61232, U10 INA210, U11 INA210, U12 INA210, U13 RN2483, U2 DRV8836DSSR, U3 DRV8836DSSR, U4 MSP432, U5 SST25VF064C, U6 DRV8836DSSR, U7 DRV8836DSSR, U8 MAX6001SOT-23, U9 INA210

Commit message: generated gerber files and pannelized pcbs
Parts:
- added BLP1, RST1: PTR1B1,27, testpad:B1,27
- added C3: 1n, SparkFun-Capacitors:0603-CAP
- added C37, C38, C39, C40, C41, C49: 100n, rcl:C0603
- added C42, C43: 12p, rcl:C0603
- added C44: 120n, rcl:C0603
- added C45: 670p, rcl:C0603
- added C46: 270p, rcl:C0603
- added C47: 10u, rcl:C0603
- added C48: 1u, rcl:C0603
- added C50: 10uF, SparkFun-Retired:EIA3216
- added C8: 100n, SparkFun-Capacitors:0603-CAP
- added JP1: (no value), pinhead:1X07
- added L3: 100uH, AS3935:COILCRAFT
- added Q3: 32.768kHz, crystal:FC-12M
- added R17, R22: 10k, rcl:R0603
- added R23, R8: 10k, resistor:R0603
- added U14: SHT21, SENSIRION-SHT21:DFN300X300X110-7N
- added U15: BMP180, SparkFun-Sensors:BMP180
- added U16: MCP3425, phMeter:SOT-23-6
- added U17: ML8511-UV-SENSORSMD, SparkFun-Sensors:ML8511
- added U18: AS3935, AS3935:16LDMLPQ
- added U19: BNO055A, BNO055:BNO055
Connections:
- new net +3V1: C37.1, C38.1, C39.1, C41.1, C44.1, C48.2, C49.1, C50.A, C8.1, JP1.1, R17.1, R22.2, U14.5, U15.2, U15.3, U16.VDD, U17.7, U18.15, U18.16, U18.5, U18.6, U18.9, U19.17, U19.28, U19.3
- new net ACCEL_IRQ: JP1.7, U19.14
- new net ACCEL_N_BOOTLD1: BLP1.TP, R22.1, U19.4
- new net ACCEL_N_RST1: R17.2, RST1.TP, U19.11
- new net GND1: C3.2, C37.2, C38.2, C39.2, C40.1, C41.2, C42.2, C43.2, C44.2, C45.2, C46.2, C47.1, C48.1, C49.2, C50.C, C8.2, JP1.2, L3.2, R23.1, R8.2, U14.2, U15.7, U16.VIN-, U16.VSS, U17.5, U18.2, U18.4, U18.7, U18.EXP, U19.10, U19.15, U19.16, U19.18, U19.2, U19.25, U19.5, U19.6
- new net LIGHTNING_IRQ: JP1.6, U18.10
- new net N$20: C3.1, U17.10
- new net N$22: U16.VIN+, U17.8
- new net N$46: C45.1, C46.1, L3.1, R23.2, U18.3
- new net N$47: C47.2, U18.1
- new net N$48: C40.2, U19.9
- new net N$53: C43.1, Q3.1, U19.26
- new net N$55: C42.1, Q3.2, U19.27
- new net SCL1: JP1.4, U14.6, U15.5, U16.SCL, U18.11, U19.19
- new net SDA1: JP1.3, U14.1, U15.6, U16.SDA, U18.13, U19.20
- new net UV_EN: JP1.5, R8.1, U17.4
Routing:
- net +3V1: track 0.00 -> 173.3 mm, vias 0 -> 2
- net SCL1: track 0.00 -> 63.4 mm, vias 0 -> 4
- net SDA1: track 0.00 -> 63.1 mm, vias 0 -> 4
- net LIGHTNING_IRQ: track 0.00 -> 54.0 mm, vias 0 -> 3
- net ACCEL_IRQ: track 0.00 -> 41.2 mm
- net UV_EN: track 0.00 -> 40.2 mm, vias 0 -> 2
- net GND1: track 0.00 -> 26.5 mm, vias 0 -> 21
- net N$46: track 0.00 -> 15.8 mm
- net N$20: track 0.00 -> 6.62 mm
- net ACCEL_N_RST1: track 0.00 -> 5.45 mm
- net N$47: track 0.00 -> 5.28 mm
- net ACCEL_N_BOOTLD1: track 0.00 -> 5.04 mm
- net N$53: track 0.00 -> 4.92 mm
- net N$55: track 0.00 -> 4.67 mm
- net N$48: track 0.00 -> 2.98 mm
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- added copper zone on layer 1, net GND1
- added copper zone on layer 16, net GND1
Other:
- board size 80 x 48 mm -> 99.2 x 60.1 mm
- board text added: "3V3 GND"
- board text added: "3V3 GND SDA SCL UV LIG ACC"
- board text added: "5V GND"
- board text added: "5V |GND|3.3V| GND |3.3V|SCL"
- board text added: "Humidity"
- board text added: "Lightning"
- board text added: "Octanis 1 weather monitor v1"
- board text added: "Orientation"
- board text added: "Pressure"
- board text added: "U3"
- board text added: "U4"
- board text added: "UV sensor"
- board text added: "www.octanis.org"
- board text removed: "3V3"
- board text removed: "5V"
- board text removed: "5V|GND|3.3V|__GND_|3.3V|SCL"
- board text removed: "GND"
