File: octanis_eps/octanis_eps_v05/octanis_eps_v05.brd (EAGLE design)
At the start: 100 x 80 mm, 106 parts, among them IC1 OPA2333DGK, Q1 N-HEXFET-2D_SOT232-, Q100 N-HEXFET-2D_SOT232-, Q2 N-HEXFET-2D_SOT232-, Q3 32.768kHz, U1 BQ24650_RVA_16, U2 TPS630250, U3 TPS630250, U4 TPS630250, U5 TPS2022D, U6 TPS61232, U8 MSP430G2544

Commit message: Added components for MPPT-charger
Parts:
- added 10UH, 10UH1: DR127, inductors:DR127
- added 5V6, 5V7: 5V-ok, adafruit:CHIPLED_0603
- added C31, C32, C37: (no value), resistor:C0805
- added C33, C34, C35, C36, C38, C39, C40: (no value), rcl:C0603
- added D1: 1N5400, diode:DO201-15
- added D2: BAS40, diode:SOT23
- added LED5_J6, LED5_J7: (no value), jumper:SJ
- added R27, R28, R30, R31, R35: (no value), rcl:R0603
- added R29: 10, rcl:R0603
- added R32, R33: 1k, rcl:R0603
- added R_SENSE2: RSENSE1, Octanis1_EPS:4PADS_RESISTOR
- added U7, U9: CSD16327Q3_DQG_8, texasinstruments:DQG8
- moved C12 432.0 mm to (69.8, 78.7)
- moved C13 432.0 mm to (69.8, 73.7)
- moved C27 432.0 mm to (69.8, 63.5)
- moved C28 432.0 mm to (69.8, 58.4)
- moved C29 432.0 mm to (69.8, 54.6)
- moved C26 432.0 mm to (69.8, 68.6)
- moved C30 432.0 mm to (69.8, 48.3)
- moved L5 432.0 mm to (69.8, 44.5)
- moved C21 352.0 mm to (63.5, 38.1)
- moved C24 352.0 mm to (63.5, 15.2)
- moved C25 352.0 mm to (63.5, 10.2)
- moved R22 352.0 mm to (63.5, 54.6)
- moved R23 352.0 mm to (63.5, 50.8)
- moved R24 352.0 mm to (63.5, 47.0)
- moved R25 352.0 mm to (63.5, 22.9)
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Connections:
- removed net BTST: U1.16
- removed net EPAD: U1.17
- removed net PH: U1.14
- removed net REGN: U1.12
- removed net VCC: U1.1
- new net N$64: R27.1, R28.2, U1.2
- new net N$65: C38.1, R35.1
- new net N$66: 5V7.A, R33.1
- new net N$67: 5V6.C, LED5_J6.2
- new net N$68: 5V7.C, LED5_J7.2
- new net N$69: 5V6.A, R32.1
- new net N$70: LED5_J6.1, U1.5
- new net N$71: LED5_J7.1, U1.3
- new net N$72: C39.1, U1.6
- new net N$73: C40.1, R29.1, U1.1
- new net N$74: D1.A, R27.2, R35.2
- new net N$75: C37.2, D1.C, R29.2, U7.5, U7.6, U7.7, U7.8
- new net N$76: 10UH1.1, C36.1, U1.14, U7.1, U7.2, U7.3, U9.5, U9.6, U9.7, U9.8
- new net N$77: C35.2, R_SENSE2.V2, U1.10
- new net N$78: C35.1, R_SENSE2.V1, U1.9
- new net N$79: 10UH1.2, R_SENSE2.I2
- new net N$80: U1.15, U7.4
- new net N$81: U1.13, U9.4
- new net N$82: C34.2, R30.1, R31.2
- new net N$83: C31.1, C32.1, C34.1, R30.2, R_SENSE2.I1
- new net N$84: C33.1, D2.1, U1.12
- new net N$85: C36.2, D2.3, U1.16
- net GND: now also C31.2, C32.2, C33.2, C37.1, C38.2, C39.2, C40.2, R28.1, R31.1, U1.17, U1.7, U9.1, U9.2, U9.3
- net VREF: no longer U1.6
