File: octanis_eps/octanis_eps_v05/octanis_eps_v05.sch (EAGLE design)
At the start: 106 parts, among them IC1 OPA2333DGK, Q1 N-HEXFET-2D_SOT232-, Q100 N-HEXFET-2D_SOT232-, Q2 N-HEXFET-2D_SOT232-, Q3 32.768kHz, U1 BQ24650_RVA_16, U2 TPS630250, U3 TPS630250, U4 TPS630250, U5 TPS2022D, U6 TPS61232, U8 MSP430G2544

Commit message: Added components for MPPT-charger
Parts:
- added 10UH, 10UH1: DR127, inductors:DR127
- added 5V6, 5V7: 5V-ok, adafruit:LEDCHIPLED_0603
- added C31, C32, C37: (no value), resistor:C-EUC0805
- added C33, C34, C35, C36, C38, C39, C40: (no value), rcl:C-EUC0603
- added D1: 1N5400, diode:1N5400
- added D2: BAS40, diode:BAS40
- added LED5_J6, LED5_J7: (no value), jumper:SJ
- added R27, R28, R30, R31, R35: (no value), rcl:R-EU_R0603
- added R29: 10, rcl:R-EU_R0603
- added R32, R33: 1k, rcl:R-EU_R0603
- added R_SENSE2: RSENSE1, Octanis1_EPS:CURRENT_RESISTOR
- added U7, U9: CSD16327Q3_DQG_8, texasinstruments:CSD16327Q3_DQG_8
Connections:
- new net N$64: R27.1, R28.2, U1.MPPSET
- new net N$65: C38.1, R35.1
- new net N$66: 5V7.A, R33.1
- new net N$67: 5V6.C, LED5_J6.2
- new net N$68: 5V7.C, LED5_J7.2
- new net N$69: 5V6.A, R32.1
- new net N$70: LED5_J6.1, U1.STAT2
- new net N$71: LED5_J7.1, U1.STAT1
- new net N$72: C39.1, U1.VREF
- new net N$73: C40.1, R29.1, U1.VCC
- new net N$74: D1.A, R27.2, R35.2
- new net N$75: C37.2, D1.C, R29.2, U7.D, U7.D_2, U7.D_3, U7.D_4
- new net N$76: 10UH1.1, C36.1, U1.PH, U7.S, U7.S_2, U7.S_3, U9.D, U9.D_2, U9.D_3, U9.D_4
- new net N$77: C35.2, R_SENSE2.V2, U1.SRP
- new net N$78: C35.1, R_SENSE2.V1, U1.SRN
- new net N$79: 10UH1.2, R_SENSE2.I2
- new net N$80: U1.HIDRV, U7.G
- new net N$81: U1.LODRV, U9.G
- new net N$82: C34.2, R30.1, R31.2
- new net N$83: C31.1, C32.1, C34.1, R30.2, R_SENSE2.I1
- new net N$84: C33.1, D2.A, U1.REGN
- new net N$85: C36.2, D2.C, U1.BTST
- net GND: now also C31.2, C32.2, C33.2, C37.1, C38.2, C39.2, C40.2, R28.1, R31.1, U1.EPAD, U1.GND, U1.TERM_EN, U9.S, U9.S_2, U9.S_3
