File: magnetic_encoder/magnetic_encoder.sch (EAGLE design)
At the start: 13 parts

Commit message: silk layer
Parts:
- renumbered U$2 to AS5600
Changed lines of the file:
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@@
 <part name="+3V3" library="supply1" deviceset="+3V3" device=""/>
 <part name="GND3" library="supply1" deviceset="GND" device=""/>
-<part name="U$2" library="austriamicrosystems" deviceset="AS5600" device=""/>
+<part name="AS5600" library="austriamicrosystems" deviceset="AS5600" device=""/>
 <part name="GND4" library="supply1" deviceset="GND" device=""/>
 <part name="+3V4" library="supply1" deviceset="+3V3" device=""/>
@@
 <instance part="+3V3" gate="G$1" x="157.48" y="66.04" rot="R270"/>
 <instance part="GND3" gate="1" x="157.48" y="58.42" rot="R90"/>
-<instance part="U$2" gate="G$1" x="99.06" y="15.24"/>
+<instance part="AS5600" gate="G$1" x="99.06" y="15.24"/>
 <instance part="GND4" gate="1" x="60.96" y="5.08"/>
 <instance part="+3V4" gate="G$1" x="78.74" y="27.94"/>
@@
 </segment>
 <segment>
-<pinref part="U$2" gate="G$1" pin="GND"/>
+<pinref part="AS5600" gate="G$1" pin="GND"/>
 <wire x1="83.82" y1="12.7" x2="78.74" y2="12.7" width="0.1524" layer="91"/>
 <wire x1="78.74" y1="12.7" x2="78.74" y2="7.62" width="0.1524" layer="91"/>
@@
 </segment>
 <segment>
-<pinref part="U$2" gate="G$1" pin="VDD5V"/>
+<pinref part="AS5600" gate="G$1" pin="VDD5V"/>
 <wire x1="83.82" y1="20.32" x2="78.74" y2="20.32" width="0.1524" layer="91"/>
 <pinref part="C4" gate="G$1" pin="2"/>
@@
 <wire x1="78.74" y1="20.32" x2="78.74" y2="25.4" width="0.1524" layer="91"/>
 <wire x1="78.74" y1="20.32" x2="78.74" y2="17.78" width="0.1524" layer="91"/>
-<pinref part="U$2" gate="G$1" pin="VDD3V3"/>
+<pinref part="AS5600" gate="G$1" pin="VDD3V3"/>
 <pinref part="C3" gate="G$1" pin="2"/>
 <wire x1="83.82" y1="17.78" x2="78.74" y2="17.78" width="0.1524" layer="91"/>
@@
 </segment>
 <segment>
-<pinref part="U$2" gate="G$1" pin="DIR"/>
+<pinref part="AS5600" gate="G$1" pin="DIR"/>
 <wire x1="114.3" y1="20.32" x2="127" y2="20.32" width="0.1524" layer="91"/>
 <label x="119.38" y="20.32" size="1.778" layer="95"/>
@@
 </segment>
 <segment>
-<pinref part="U$2" gate="G$1" pin="SDA"/>
+<pinref part="AS5600" gate="G$1" pin="SDA"/>
 <wire x1="114.3" y1="15.24" x2="127" y2="15.24" width="0.1524" layer="91"/>
 <label x="119.38" y="15.24" size="1.778" layer="95"/>
@@
 </segment>
 <segment>
-<pinref part="U$2" gate="G$1" pin="SCL"/>
+<pinref part="AS5600" gate="G$1" pin="SCL"/>
 <wire x1="114.3" y1="17.78" x2="127" y2="17.78" width="0.1524" layer="91"/>
 <label x="119.38" y="17.78" size="1.778" layer="95"/>
@@
 </segment>
 <segment>
-<pinref part="U$2" gate="G$1" pin="OUT"/>
+<pinref part="AS5600" gate="G$1" pin="OUT"/>
 <wire x1="83.82" y1="15.24" x2="78.74" y2="15.24" width="0.1524" layer="91"/>
 <wire x1="78.74" y1="15.24" x2="76.2" y2="15.24" width="0.1524" layer="91"/>
@@
 <net name="CS/PGO" class="0">
 <segment>
-<pinref part="U$2" gate="G$1" pin="PGO"/>
+<pinref part="AS5600" gate="G$1" pin="PGO"/>
 <wire x1="114.3" y1="12.7" x2="127" y2="12.7" width="0.1524" layer="91"/>
 <label x="119.38" y="12.7" size="1.778" layer="95"/>
