File: octanis_eps/v0.4_second_run/octanis_eps_v04.sch (EAGLE design)
At the start: 107 parts, among them IC1 OPA2333DGK, IC100 OPA2333DGK, IC101 OPA347, IC2 OPA2333DGK, Q1 N-HEXFET-2D_SOT232-, Q100 N-HEXFET-2D_SOT232-, Q2 N-HEXFET-2D_SOT232-, Q3 FC-12M

Commit message: minor eps changes. stencil laser cut files for v0.6 added
Parts:
- C13: value 4.7u -> 4.7uF
- C14, C4: value 22u -> 22uF
- C3: value 10u -> 10uF
- C8: value 4.7p -> 4.7pF
- C9: value 470p -> 470pF
- RSENSE1: value RSENSE2 -> 10m
- RSENSE2: value RSENSE3 -> 50m
- R_SENSE1: value RSENSE1 -> 10m
Changed lines of the file:
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@@
 <grid distance="0.1" unitdist="inch" unit="inch" style="lines" multiple="1" display="no" altdistance="0.01" altunitdist="inch" altunit="inch"/>
 <layers>
-<layer number="1" name="Top" color="4" fill="1" visible="yes" active="no"/>
-<layer number="16" name="Bottom" color="1" fill="1" visible="yes" active="no"/>
-<layer number="17" name="Pads" color="2" fill="1" visible="yes" active="no"/>
-<layer number="18" name="Vias" color="2" fill="1" visible="yes" active="no"/>
-<layer number="19" name="Unrouted" color="6" fill="1" visible="yes" active="no"/>
-<layer number="20" name="Dimension" color="15" fill="1" visible="yes" active="no"/>
-<layer number="21" name="tPlace" color="7" fill="1" visible="yes" active="no"/>
-<layer number="22" name="bPlace" color="7" fill="1" visible="yes" active="no"/>
-<layer number="23" name="tOrigins" color="15" fill="1" visible="yes" active="no"/>
-<layer number="24" name="bOrigins" color="15" fill="1" visible="yes" active="no"/>
-<layer number="25" name="tNames" color="7" fill="1" visible="yes" active="no"/>
-<layer number="26" name="bNames" color="7" fill="1" visible="yes" active="no"/>
-<layer number="27" name="tValues" color="7" fill="1" visible="yes" active="no"/>
-<layer number="28" name="bValues" color="7" fill="1" visible="yes" active="no"/>
+<layer number="1" name="Top" color="4" fill="1" visible="no" active="no"/>
+<layer number="16" name="Bottom" color="1" fill="1" visible="no" active="no"/>
+<layer number="17" name="Pads" color="2" fill="1" visible="no" active="no"/>
+<layer number="18" name="Vias" color="2" fill="1" visible="no" active="no"/>
+<layer number="19" name="Unrouted" color="6" fill="1" visible="no" active="no"/>
+<layer number="20" name="Dimension" color="15" fill="1" visible="no" active="no"/>
+<layer number="21" name="tPlace" color="7" fill="1" visible="no" active="no"/>
+<layer number="22" name="bPlace" color="7" fill="1" visible="no" active="no"/>
+<layer number="23" name="tOrigins" color="15" fill="1" visible="no" active="no"/>
+<layer number="24" name="bOrigins" color="15" fill="1" visible="no" active="no"/>
+<layer number="25" name="tNames" color="7" fill="1" visible="no" active="no"/>
+<layer number="26" name="bNames" color="7" fill="1" visible="no" active="no"/>
+<layer number="27" name="tValues" color="7" fill="1" visible="no" active="no"/>
+<layer number="28" name="bValues" color="7" fill="1" visible="no" active="no"/>
 <layer number="29" name="tStop" color="7" fill="3" visible="no" active="no"/>
 <layer number="30" name="bStop" color="7" fill="6" visible="no" active="no"/>
@@
 <layer number="35" name="tGlue" color="7" fill="4" visible="no" active="no"/>
 <layer number="36" name="bGlue" color="7" fill="5" visible="no" active="no"/>
-<layer number="37" name="tTest" color="7" fill="1" visible="yes" active="no"/>
-<layer number="38" name="bTest" color="7" fill="1" visible="yes" active="no"/>
+<layer number="37" name="tTest" color="7" fill="1" visible="no" active="no"/>
+<layer number="38" name="bTest" color="7" fill="1" visible="no" active="no"/>
 <layer number="39" name="tKeepout" color="4" fill="11" visible="no" active="no"/>
 <layer number="40" name="bKeepout" color="1" fill="11" visible="no" active="no"/>
@@
 <layer number="44" name="Drills" color="7" fill="1" visible="no" active="no"/>
 <layer number="45" name="Holes" color="7" fill="1" visible="no" active="no"/>
-<layer number="46" name="Milling" color="3" fill="1" visible="yes" active="no"/>
-<layer number="47" name="Measures" color="7" fill="1" visible="yes" active="no"/>
-<layer number="48" name="Document" color="7" fill="1" visible="yes" active="no"/>
-<layer number="49" name="Reference" color="7" fill="1" visible="yes" active="no"/>
-<layer number="50" name="dxf" color="7" fill="1" visible="yes" active="no"/>
-<layer number="51" name="tDocu" color="7" fill="1" visible="yes" active="no"/>
-<layer number="52" name="bDocu" color="7" fill="1" visible="yes" active="no"/>
-<layer number="53" name="tGND_GNDA" color="7" fill="9" visible="yes" active="no"/>
-<layer number="54" name="bGND_GNDA" color="1" fill="9" visible="yes" active="no"/>
-<layer number="56" name="wert" color="7" fill="1" visible="yes" active="no"/>
+<layer number="46" name="Milling" color="3" fill="1" visible="no" active="no"/>
+<layer number="47" name="Measures" color="7" fill="1" visible="no" active="no"/>
+<layer number="48" name="Document" color="7" fill="1" visible="no" active="no"/>
+<layer number="49" name="Reference" color="7" fill="1" visible="no" active="no"/>
+<layer number="50" name="dxf" color="7" fill="1" visible="no" active="no"/>
+<layer number="51" name="tDocu" color="7" fill="1" visible="no" active="no"/>
+<layer number="52" name="bDocu" color="7" fill="1" visible="no" active="no"/>
+<layer number="53" name="tGND_GNDA" color="7" fill="9" visible="no" active="no"/>
+<layer number="54" name="bGND_GNDA" color="1" fill="9" visible="no" active="no"/>
+<layer number="56" name="wert" color="7" fill="1" visible="no" active="no"/>
 <layer number="90" name="Modules" color="5" fill="1" visible="yes" active="yes"/>
 <layer number="91" name="Nets" color="2" fill="1" visible="yes" active="yes"/>
@@
 <part name="R29" library="rcl" deviceset="R-EU_" device="R0603" value="200k"/>
 <part name="R6" library="rcl" deviceset="R-EU_" device="R0603" value="1M"/>
-<part name="C13" library="rcl" deviceset="C-EU" device="C1206" value="4.7u"/>
-<part name="C9" library="rcl" deviceset="C-EU" device="C0603" value="470p"/>
-<part name="C14" library="rcl" deviceset="C-EU" device="C0603" value="22u"/>
+<part name="C13" library="rcl" deviceset="C-EU" device="C1206" value="4.7uF"/>
+<part name="C9" library="rcl" deviceset="C-EU" device="C0603" value="470pF"/>
+<part name="C14" library="rcl" deviceset="C-EU" device="C0603" value="22uF"/>
 <part name="R12" library="rcl" deviceset="R-EU_" device="R0603" value="82k"/>
-<part name="C3" library="rcl" deviceset="C-EU" device="C1206" value="10u"/>
-<part name="C4" library="rcl" deviceset="C-EU" device="C1206" value="22u"/>
-<part name="C8" library="rcl" deviceset="C-EU" device="C0603" value="4.7p"/>
+<part name="C3" library="rcl" deviceset="C-EU" device="C1206" value="10uF"/>
+<part name="C4" library="rcl" deviceset="C-EU" device="C1206" value="22uF"/>
+<part name="C8" library="rcl" deviceset="C-EU" device="C0603" value="4.7pF"/>
 <part name="U$6" library="Octanis1_EPS" deviceset="LTC3402" device=""/>
 <part name="U$4" library="Octanis1_EPS" deviceset="TPS62086" device=""/>
@@
 <part name="SUPPLY55" library="supply2" deviceset="VCC" device=""/>
 <part name="SUPPLY56" library="supply2" deviceset="VCC" device=""/>
-<part name="R_SENSE1" library="Octanis1_EPS" deviceset="CURRENT_RESISTOR" device="" value="RSENSE1"/>
-<part name="RSENSE1" library="Octanis1_EPS" deviceset="CURRENT_RESISTOR" device="" value="RSENSE2"/>
-<part name="RSENSE2" library="Octanis1_EPS" deviceset="CURRENT_RESISTOR" device="" value="RSENSE3"/>
+<part name="R_SENSE1" library="Octanis1_EPS" deviceset="CURRENT_RESISTOR" device="" value="10m"/>
+<part name="RSENSE1" library="Octanis1_EPS" deviceset="CURRENT_RESISTOR" device="" value="10m"/>
+<part name="RSENSE2" library="Octanis1_EPS" deviceset="CURRENT_RESISTOR" device="" value="50m"/>
 <part name="BT_CHG" library="pinhead" deviceset="PINHD-1X1" device=""/>
 <part name="DSP_CMD" library="pinhead" deviceset="PINHD-1X1" device=""/>
