File: external_weather_strip/external_strip_v3.sch (EAGLE design)
At the start: 31 parts, among them Q1 32.768kHz, U1 BMP180, U2 SHT21, U3 ML8511-UV-SENSORSMD, U4 MCP3425, U5 BNO055A, U6 AS3935

Commit message: weather strip v3. revised mainboard v1
Parts:
- removed JP1: (no value), pinhead:PINHD-1X7
- removed RST: PTR1B1,27, testpad:PTR1B1,27
- removed U1: BMP180, SparkFun-Sensors:BMP180
- added C9B: 10n, rcl:C-EUC0603
- added IC1: BMP280, we-sensor:BMP280
- added JP2: (no value), Headerlibrary:PINHD-1X8
- added L2: 100uH, AS3935:COILCRAFT
- added LED5_J: (no value), jumper:SJ
- added ON: 3V3_ok, adafruit:LEDCHIPLED_0603
- added R101: 2k, rcl:R-EU_R0603
- added TP1: TEST-POINT3, SparkFun:TEST-POINT3
- added U7: AS3935, AS3935:AS3935
- C9A: value 120n -> 100n
- L1: value 100uH -> (none); device AS3935:COILCRAFT -> dp_devices:FERRITE-0603
- U5: value BNO055A -> LM4132-2.048V; device BNO055:BNO055A -> SparkFun:LM4128-2.5VREF
- U6: value AS3935 -> BNO055A; device AS3935:AS3935 -> BNO055:BNO055A
- renumbered C9 to C9A
Connections:
- new net AVCC: C16.+, C4.1, C6.1, L1.2, U3.VDD, U4.VDD
- new net N$4: LED5_J.2, ON.C
- new net N$6: U4.VIN-, U5.VOUT
- new net N$8: ON.A, R101.1
- net +3V3: now also C9B.1, IC1.CSB, IC1.SDO, IC1.VCCIO, JP2.1, L1.1, R101.2, TP1.1, U5.VIN, U6.COM3, U6.VDDIO, U7.ADD0, U7.ADD1, U7.SI, U7.VDD, U7.VREG; no longer C16.+, C4.1, C6.1, JP1.1, U1.VDD, U1.VDDIO, U3.VDD, U4.VDD, U5.COM3, U5.VDD, U5.VDDIO, U6.ADD0, U6.ADD1, U6.SI, U6.VREG
- net ACCEL_IRQ: now also JP2.7, U6.INT; no longer JP1.7, U5.INT
- net ACCEL_N_BOOTLD: now also U6.BOOT_LOAD_PIN; no longer U5.BOOT_LOAD_PIN
- net ACCEL_N_RST: now also U6.RESET; no longer RST.TP, U5.RESET
- net GND: now also C9B.2, IC1.GND@1, IC1.GND@2, JP2.2, JP2.8, L2.2, LED5_J.1, U6.COM2, U6.GNDIO, U6.PIN10, U6.PIN15, U6.PIN16, U6.PS0, U6.PS1, U7.EN_VREG, U7.EXPAD, U7.GND, U7.INN; no longer JP1.2, L1.2, U1.GND, U4.VIN-, U5.COM2, U5.GNDIO, U5.PIN10, U5.PIN15, U5.PIN16, U5.PS0, U5.PS1, U6.EN_VREG, U6.EXPAD, U6.INN
- net LIGHTNING_IRQ: now also JP2.6, U7.IRQ; no longer JP1.6, U6.IRQ
- net N$18: now also U6.CAP; no longer U5.CAP
- net N$19: now also U6.XIN32; no longer U5.XIN32
- net N$2: now also U7.ACG; no longer U6.ACG
- net N$5: now also L2.1, U7.INP; no longer L1.1, U6.INP
- net N$73: now also U6.XOUT32; no longer U5.XOUT32
- net SCL: now also IC1.SCK, JP2.4, U6.COM1, U7.I2CL/SCL; no longer JP1.4, U1.SCL, U5.COM1, U6.I2CL/SCL
- net SDA: now also IC1.SDI, JP2.3, U6.COM0, U7.I2CD/MOSI; no longer JP1.3, U1.SDA, U5.COM0, U6.I2CD/MOSI
- net UV_EN: now also JP2.5, U5.EN; no longer JP1.5
Other:
- moved on the sheet: C4
