File: external_weather_strip/external_strip_v3.brd (EAGLE design)
At the start: 40 x 30 mm, 37 parts, among them IC1 BMP280, Q1 32.768kHz, U2 SHT21, U3 ML8511-UV-SENSORSMD, U4 MCP3425, U5 LM4132-2.048V, U6 BNO055A, U7 AS3935

Commit message: created final gerber files
Routing:
- net GND: track 37.0 -> 39.3 mm
Other:
- board text added: "3V3_GND_SDA_SCL_UV_LIG_ACC_GND"
- board text removed: "3V3 GND SDA SCL UV LIG ACC GND"
Changed lines of the file:
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@@
 <text x="24.765" y="10.795" size="1.016" layer="27">MCP3425</text>
 <text x="27.94" y="6.35" size="1.016" layer="27">ML8511 </text>
-<text x="-0.1524" y="7.1336" size="0.8128" layer="25" rot="R90">3V3 GND SDA SCL  UV  LIG  ACC GND</text>
+<text x="-0.1524" y="6.3716" size="0.8128" layer="25" rot="R90">3V3_GND_SDA_SCL_UV_LIG_ACC_GND</text>
 <text x="6.096" y="18.5928" size="0.8128" layer="25" font="fixed">Octanis 1 weather board v3</text>
 <text x="6.096" y="17.3736" size="0.8128" layer="25" font="fixed">www.octanis.org</text>
@@
 <wire x1="28.718" y1="4.475" x2="28.688" y2="4.445" width="1.27" layer="16"/>
 <wire x1="28.688" y1="4.445" x2="26.67" y2="4.445" width="1.27" layer="16"/>
-<wire x1="25.6952" y1="26.9394" x2="25.6952" y2="25.6394" width="0" layer="19" extent="1-1"/>
 <via x="-0.4064" y="6.0198" extent="1-16" drill="0.3048"/>
 <via x="-0.7112" y="28.575" extent="1-16" drill="0.3048"/>
 <via x="-0.4064" y="4.4958" extent="1-16" drill="0.3048"/>
+<wire x1="25.6952" y1="25.6394" x2="25.659" y2="25.6032" width="0.4064" layer="1"/>
+<wire x1="25.659" y1="25.6032" x2="24.0792" y2="25.6032" width="0.4064" layer="1"/>
+<wire x1="24.0792" y1="25.6032" x2="23.718" y2="25.9644" width="0.4064" layer="1"/>
+<wire x1="23.718" y1="25.9644" x2="23.5952" y2="25.9644" width="0.4064" layer="1"/>
 </signal>
 <signal name="UV_EN">
