File: external_weather_strip/external_strip_v4.sch (EAGLE design)
At the start: 37 parts, among them IC1 BMP280, Q1 32.768kHz, U2 SHT21, U3 ML8511-UV-SENSORSMD, U4 MCP3425, U5 LM4132-2.048V, U6 BNO055A, U7 AS3935

Commit message: finalized silkscreen, generated Gerber files for EPS v2; replaced UV sensor in weather board, generated gerber files for v4
Parts:
- removed C16: 10uF, SparkFun-Retired:10UF-TANT
- removed C4: 100n, SparkFun-Capacitors:0.1UF-25V(+80/-20%)(0603)
- removed C5: 1n, SparkFun-Capacitors:1NF/1000PF-50V-10%(0603)
- removed L1: (no value), dp_devices:FERRITE-0603
- removed U6: BNO055A, BNO055:BNO055A
- removed U7: AS3935, AS3935:AS3935
- added R5: 5k1, rcl:R-EU_R0603
- R1: device resistor:R-EU_R0603 -> rcl:R-EU_R0603
- U3: value ML8511-UV-SENSORSMD -> SI1133; device SparkFun-Sensors:ML8511-UV-SENSORSMD -> Octanis1:SI1133
- U4: value MCP3425 -> BNO055A; device phMeter:MCP3425 -> BNO055:BNO055A
- U5: value LM4132-2.048V -> AS3935; device SparkFun:LM4128-2.5VREF -> AS3935:AS3935
- renumbered IC1 to U1
Connections:
- removed net AVCC: C16.+, C4.1, C6.1, L1.2, U3.VDD, U4.VDD
- removed net N$1: U3.OUT, U4.VIN+
- removed net N$3: C5.1, U3.TR
- removed net N$6: U4.VIN-, U5.VOUT
- removed net UV_EN: JP2.5, R1.1, U3.EN, U5.EN
- new net N$9: R1.1, U3.AD, U3.RUP1, U3.RUP2
- new net UV_IRQ: JP2.5, R5.2, U3.INT
- net +3V3: now also C6.1, R1.2, R5.1, U3.VDD, U4.COM3, U4.VDD, U4.VDDIO, U5.ADD0, U5.ADD1, U5.SI, U5.VDD, U5.VREG; no longer L1.1, U5.VIN, U6.COM3, U6.VDD, U6.VDDIO, U7.ADD0, U7.ADD1, U7.SI, U7.VDD, U7.VREG
- net ACCEL_IRQ: now also U4.INT; no longer U6.INT
- net ACCEL_N_BOOTLD: now also U4.BOOT_LOAD_PIN; no longer U6.BOOT_LOAD_PIN
- net ACCEL_N_RST: now also U4.RESET; no longer U6.RESET
- net GND: now also U4.COM2, U4.GND, U4.GNDIO, U4.PIN10, U4.PIN15, U4.PIN16, U4.PS0, U4.PS1, U5.EN_VREG, U5.EXPAD, U5.INN; no longer C16.-, C4.2, C5.2, R1.2, U4.VSS, U6.COM2, U6.GND, U6.GNDIO, U6.PIN10, U6.PIN15, U6.PIN16, U6.PS0, U6.PS1, U7.EN_VREG, U7.EXPAD, U7.GND, U7.INN
- net LIGHTNING_IRQ: now also U5.IRQ; no longer U7.IRQ
- net N$18: now also U4.CAP; no longer U6.CAP
- net N$19: now also U4.XIN32; no longer U6.XIN32
- net N$2: now also U5.ACG; no longer U7.ACG
- net N$5: now also U5.INP; no longer U7.INP
- net N$73: now also U4.XOUT32; no longer U6.XOUT32
- net SCL: now also U3.SCL, U4.COM1, U5.I2CL/SCL; no longer U4.SCL, U6.COM1, U7.I2CL/SCL
- net SDA: now also U3.SDA, U4.COM0, U5.I2CD/MOSI; no longer U4.SDA, U6.COM0, U7.I2CD/MOSI
Other:
- moved on the sheet: C6, R1
