File: octanis_eps/v1.0/octanis_eps_v1.sch (EAGLE design)
At the start: 155 parts, among them IC1 OPA2333DGK, Q1 32.768kHz, Q100 BSS123, Q2 BSC0901NS, U1 CSD16327Q3_DQG_8, U10 CSD16327Q3_DQG_8, U11 CSD16327Q3_DQG_8, U12 TPS630250YFFT, U15 MSP430FR5969, U2 CSD16327Q3_DQG_8, U3 CSD16327Q3_DQG_8, U5 TPS2022D, U6 TPS630250YFFT, U7 TPS630250YFFT, U8 TPS61232, U9 BQ24650_RVA_16

Commit message: reworked silkscreen
Parts:
- removed 6.8UH: DR127, inductors:DR127
- removed C100, C_IC1: 100nF, rcl:C-EUC0603
- removed C101: 1uF, rcl:C-EUC0603
- removed C102, C103: 22uF, resistor:C-EUC0805
- removed C104: 10uF, resistor:C-EUC0805
- removed IC1: OPA2333DGK, linear:OPA2333DGK
- removed JP8: (no value), Headerlibrary:PINHD-2X6
- removed L100: 1uH, Coilcraft:XFL4020
- removed R100, R101: (no value), rcl:R-EU_R0603
- removed R102, R103: 1M, rcl:R-EU_R0603
- removed R104: 1M, resistor:R-EU_R0603
- removed U$1: TPS61088, texasinstruments:TPS61088
- removed U$2, U$3: INA213, Octanis1_EPS:INA213
- removed U$5: MIC5019, Octanis1_EPS:MIC5019
- removed U15: MSP430FR5969, chips:MSP430FR5969
- added C41, C42, C44: 10uF, resistor:C-EUC0805
- added C43: 47uF Tantal, rcl:C-EUC1210
- added C45: 100nF, rcl:C-EUC0603
- added C46: 47nF, rcl:C-EUC0603
- added JP1, VCC_GND: (no value), Headerlibrary:PINHD-1X2
- added L5: 1uH, Coilcraft:XFL4020
- added L6: 1.5uH, Coilcraft:XFL4020
- added Q3, Q5, Q6: CSD16327Q3_DQG_8, texasinstruments:CSD16327Q3_DQG_8
- added Q7: BSC0901NS, transistor-power:BSC340N08NS3G
- added R44: 100k, resistor:R-EU_R0603
- added R45: 150-220k, resistor:R-EU_R0603
- added R46: 56k, resistor:R-EU_R0603
- added R47: 470k, resistor:R-EU_R0603
- added R48: dnp, resistor:R-EU_R0603
- added U4: TPS630250YFFT, texasinstruments:TPS630250YFFT
- added X1: 32.768kHz, microcrystal:MS3V-T1R
- C10: value 10uF -> 1.5uF; device resistor:C-EUC0805 -> rcl:C-EUC0603
- C13: value 10nF -> 10uF; device rcl:C-EUC0603 -> resistor:C-EUC0805
- C14, C38: value 10uF -> 22uF
- C15: value 100nF -> 22uF; device rcl:C-EUC0603 -> resistor:C-EUC0805
- C16, C18: value 22uF -> 1uF; device resistor:C-EUC0805 -> rcl:C-EUC0603
- C17, C29, C5: value 22uF -> 100nF; device resistor:C-EUC0805 -> rcl:C-EUC0603
- C19: value 22uF -> 10uF; device rcl:C-EUC0603 -> resistor:C-EUC0805
- C2, C8: value 1.5uF -> 100nF
- C20: value 1uF -> 10nF
- C21: value 1u -> 22uF; device rcl:C-EUC0603 -> resistor:C-EUC0805
- C22: value 2.2uF -> 22uF; device rcl:C-EUC0603 -> resistor:C-EUC0805
- C23: value 2.2uF -> 10uF; device rcl:C-EUC0603 -> resistor:C-EUC0805
- C24: value 150pF -> 22uF; device rcl:C-EUC0603 -> resistor:C-EUC0805
- C25: value 4.7nF -> 22uF; device rcl:C-EUC0603 -> resistor:C-EUC0805
- C26: value 22pF -> 22uF; device rcl:C-EUC0603 -> resistor:C-EUC0805
- C27: value 1uF -> 2.2uF
- C28: value 22uF -> 1u; device resistor:C-EUC0805 -> rcl:C-EUC0603
- C3: value 100nF -> 1.5uF
- C30: value 22uF -> 22pF; device resistor:C-EUC0805 -> rcl:C-EUC0603
- C31: value 100nF -> 22uF
- C32: value 10uF -> 100nF; device resistor:C-EUC0805 -> rcl:C-EUC0603
- C33: value 47uF Tantal -> 2.2uF; device rcl:C-EUC1210 -> rcl:C-EUC0603
- C34: value 10uF -> 1uF; device resistor:C-EUC0805 -> rcl:C-EUC0603
- C35: value 100nF -> 150pF
- C36: value 47nF -> 22uF; device rcl:C-EUC0603 -> resistor:C-EUC0805
- C37: value 10uF -> 4.7nF; device resistor:C-EUC0805 -> rcl:C-EUC0603
- C39: value 12pF -> 22uF; device rcl:C-EUC0603 -> resistor:C-EUC0805
- C4: value 100nF -> 10uF; device rcl:C-EUC0603 -> rcl:CPOL-EUA/3216-18R
- C40: value 12pF -> 10uF; device rcl:C-EUC0603 -> resistor:C-EUC0805
- C6: value 22uF -> 12pF; device resistor:C-EUC0805 -> rcl:C-EUC0603
- C7: value 10uF -> 12pF; device rcl:CPOL-EUA/3216-18R -> rcl:C-EUC0603
- JP2: device Headerlibrary:PINHD-1X2 -> Headerlibrary:PINHD-2X6
- L4: value 1.5uH -> DR127_6u8; device Coilcraft:XFL4020 -> inductors:DR127
- Q1: value 32.768kHz -> CSD16327Q3_DQG_8; device microcrystal:MS3V-T1R -> texasinstruments:CSD16327Q3_DQG_8
- Q2: value BSC0901NS -> CSD16327Q3_DQG_8; device transistor-power:BSC340N08NS3G -> texasinstruments:CSD16327Q3_DQG_8
- R1: value 1k -> 10k
- R10, R18, R22: value 200k -> 1k
- R14: value 1k -> 1.5k
- R15: value 1.5k -> 4.7k
- R16: value 4.7k -> 1k
- R17, R21, R32: value 100k -> 1M
- R19: value 10k -> 1M
- R2, R25: value 1k -> 200k
- R20: value 100k -> 1k
- R24: value 1M -> 1k; device resistor:R-EU_R0603 -> rcl:R-EU_R0603
- R26: value 1k -> 1M; device rcl:R-EU_R0603 -> resistor:R-EU_R0603
- R29: value 4k7 -> (none)
- R3: value 1k -> 100k
- R30: value 1M -> 4k7
- R33: value 100k -> (none)
- R34: value 2.2M -> 100k
- R35: device resistor:R-EU_R0603 -> rcl:R-EU_R0603
- R36: value 56k -> 1M; device resistor:R-EU_R0603 -> rcl:R-EU_R0603
- R37: value 150-220k -> 1M; device resistor:R-EU_R0603 -> rcl:R-EU_R0603
- R38: value 470k -> 1M
- R39: value 47k -> 2; device resistor:R-EU_R0603 -> rcl:R-EU_R2010
- R4, R6, R8: value 1M -> 100k
- R41: value 2 -> 2.2M; device rcl:R-EU_R2010 -> rcl:R-EU_R0603
- R42: value dnp -> 1M; device resistor:R-EU_R0603 -> rcl:R-EU_R0603
- R43: value 1M -> 47k; device rcl:R-EU_R0603 -> resistor:R-EU_R0603
- R9: value 100k -> 200k
- RS1: value RSENSE1 10mOhm -> 10m
- RS2: value RSENSE2 -> 50m
- RS3: value RSENSE1 -> 50m
- RT2: value 8501 -> 2723
- RT4: value 2723 -> 8501
- U1: value CSD16327Q3_DQG_8 -> MSP430FR5969; device texasinstruments:CSD16327Q3_DQG_8 -> chips:MSP430FR5969
- U10: value CSD16327Q3_DQG_8 -> INA213; device texasinstruments:CSD16327Q3_DQG_8 -> Octanis1_EPS:INA213
- U11: value CSD16327Q3_DQG_8 -> MIC5019; device texasinstruments:CSD16327Q3_DQG_8 -> Octanis1_EPS:MIC5019
- U12: value TPS630250YFFT -> TPS61088; device texasinstruments:TPS630250YFFT -> texasinstruments:TPS61088
- U2: value CSD16327Q3_DQG_8 -> OPA2333DGK; device texasinstruments:CSD16327Q3_DQG_8 -> linear:OPA2333DGK
- U3: value CSD16327Q3_DQG_8 -> TPS2022D; device texasinstruments:CSD16327Q3_DQG_8 -> Octanis1_EPS:TPS2022D
- U5: value TPS2022D -> BQ24650_RVA_16; device Octanis1_EPS:TPS2022D -> octanis_eps_v05:BQ24650_RVA_16
- U7: value TPS630250YFFT -> TPS61232; device texasinstruments:TPS630250YFFT -> texasinstruments:TPS61232
- U8: value TPS61232 -> TPS630250YFFT; device texasinstruments:TPS61232 -> texasinstruments:TPS630250YFFT
- U9: value BQ24650_RVA_16 -> INA213; device octanis_eps_v05:BQ24650_RVA_16 -> Octanis1_EPS:INA213
- renumbered FERRITE to LF2, FERRITE1 to LF3, FERRITE2 to LF1, J1 to J107, J2 to J106, J3 to J105, J4 to J104, J5 to J103, J6 to J102, J7 to J101, J8 to J100, JP7 to DIGITAL, Q100 to Q4, RSENSE1 to RS2, R_SENSE1 to RS1, R_SENSE2 to RS3
Connections:
- net +12V: now also C34.2, C36.2, C38.2, C39.2, R47.2, U12.VOUT1, U12.VOUT2, U12.VOUT3; no longer C27.2, C28.2, C29.2, C30.2, R38.2, U$1.VOUT1, U$1.VOUT2, U$1.VOUT3
- net +3V3: now also C11.1, C12.1, C4.+, R1.2, R26.2, U1.DVCC, U3.IN1, U3.IN2, U6.FB, U6.VOUT, U6.VOUT_2, U6.VOUT_3, VCC_GND.1; no longer C4.1, C6.1, C7.+, R19.2, R24.2, U12.FB, U12.VOUT, U12.VOUT_2, U12.VOUT_3, U15.DVCC, U5.IN1, U5.IN2
- net +3V3_1: now also C25.1, C26.1, U8.FB, U8.VOUT, U8.VOUT_2, U8.VOUT_3; no longer C11.1, C12.1, U6.FB, U6.VOUT, U6.VOUT_2, U6.VOUT_3
- net +3V3_2: now also C14.1, C15.1, U4.FB, U4.VOUT, U4.VOUT_2, U4.VOUT_3; no longer C102.1, C103.1, U7.FB, U7.VOUT, U7.VOUT_2, U7.VOUT_3
- net +3V3_M: now also U3.OUT1, U3.OUT2, U3.OUT3; no longer U5.OUT1, U5.OUT2, U5.OUT3
- net +5V: now also C21.1, C22.1, C24.1, R37.2, U7.FB, U7.VOUT; no longer C16.1, C17.1, C18.1, R28.2, U8.FB, U8.VOUT
- net A4_EXT: now also JP2.11, RT2.2, U1.P1.4/TB0.1/UCA0STE/A4/C4; no longer JP8.11, RT3.2, U15.P1.4/TB0.1/UCA0STE/A4/C4
- net A5_EXT: now also JP2.9, RT1.2, U1.P1.5/TB0.2/UCA0CLK/A5/C5; no longer JP8.9, RT4.2, U15.P1.5/TB0.2/UCA0CLK/A5/C5
- net AGND: now also C10.1, C3.1, C8.2, JP2.10, JP2.12, JP2.2, JP2.4, JP2.6, JP2.8, R2.2, R3.1, R6.1, R9.2, U1.AVSS, U10.GND, U10.REF, U2P.V-, U9.GND, U9.REF; no longer C3.2, C8.1, C_IC1.1, IC1P.V-, JP8.10, JP8.12, JP8.2, JP8.4, JP8.6, JP8.8, R10.2, R18.2, R20.1, R21.1, U$2.GND, U$2.REF, U$3.GND, U$3.REF, U15.AVSS
- net AVCC: now also C8.1, RT1.1, RT2.1, U1.AVCC; no longer C3.1, RT3.1, RT4.1, U15.AVCC
- net AVCC1: now also U10.VCC, U9.VCC; no longer U$2.VCC, U$3.VCC
- net AVCC2: now also C2.2, U2P.V+; no longer C_IC1.2, IC1P.V+
- net A_EXT1: now also JP2.7, U1.P4.0/A8; no longer JP8.7, U15.P4.0/A8
- net A_EXT2: now also JP2.5, U1.P4.1/A9; no longer JP8.5, U15.P4.1/A9
- net A_EXT3: now also JP2.3, U1.P4.2/A10; no longer JP8.3, U15.P4.2/A10
- net A_EXT4: now also JP2.1, U1.P4.3/A11; no longer JP8.1, U15.P4.3/A11
- net BAT_11V: now also C43.1, C44.1, C45.1, L6.1, Q7G$1.S, U12.EN, U12.VIN; no longer C33.1, C34.1, C35.1, L4.1, Q2G$1.S, U$1.EN, U$1.VIN
- net BAT_OUT: now also C13.1, C23.1, C31.1, L5.1, Q7G$1.D, U11.VDD, U4.VIN, U4.VINA, U4.VIN_2, U4.VIN_3, U6.EN, U8.VINA, U8.VIN_2, U8.VIN_3; no longer C10.1, C104.1, C14.1, L3.1, Q2G$1.D, U$5.VDD, U12.EN, U12.VIN, U12.VINA, U12.VIN_2, U12.VIN_3, U7.VINA, U7.VIN_2, U7.VIN_3
- net EN_12V: now also R42.2, U1.P3.0/A12/C12, U11.IN; no longer R43.2, U$5.IN, U15.P3.0/A12/C12
- net EN_3V3_1: now also R38.1, U1.P3.3/A15/C15, U8.EN; no longer R27.1, U15.P3.3/A15/C15, U6.EN
- net EN_3V3_2: now also R27.1, U1.P4.7, U4.EN; no longer R104.1, U15.P4.7, U7.EN
- net EN_3V3_M: now also R26.1, U1.P3.2/A14/C14, U3.EN; no longer R24.1, U15.P3.2/A14/C14, U5.EN
- net EN_5V: now also R36.2, U1.P3.1/A13/C13, U7.EN; no longer R30.2, U15.P3.1/A13/C13, U8.EN
- net EN_HEAT1: now also R16.2, R17.1, U1.PJ.0/TDO; no longer R3.2, R4.1, U15.PJ.0/TDO
- net EN_HEAT2: now also R18.2, R19.1, U1.PJ.1/TDI; no longer R5.2, R6.1, U15.PJ.1/TDI
- net EN_HEAT3: now also R20.2, R21.1, U1.PJ.2/TMS; no longer R7.2, R8.1, U15.PJ.2/TMS
- net EN_SC: now also R28.1, R32.2, U1.P3.4/TB0.3; no longer R102.1, R103.2, U15.P3.4/TB0.3
- net GND: now also C15.2, C26.2, C27.2, C28.2, C31.2, C34.1, C36.1, C38.1, C4.-, C41.2, C42.2, C43.2, C44.2, C45.2, C46.2, C6.1, C7.1, Q1.S, Q1.S_2, Q1.S_3, Q2.S, Q2.S_2, Q2.S_3, Q3.S, Q3.S_2, Q3.S_3, Q6.S, Q6.S_2, Q6.S_3, R17.2, R19.2, R21.2, R32.1, R34.1, R38.2, R42.1, R44.1, R46.1, R48.2, RT4.2, U1.DVSS, U1.VSS_QFN, U11.GND, U12.AGND, U3.GND, U4.GND, U4.PFM_PWM, U4.PGND, U4.PGND_2, U4.PGND_3, U5.EPAD, U5.TERM_EN, U7.GND1, U7.GND2, U7.GND3, U7.GND4, U7.GND5, U8.PFM_PWM, U8.PGND, U8.PGND_2, U8.PGND_3, VCC_GND.2, X1.GND; no longer C10.2, C101.2, C102.2, C103.2, C104.2, C17.2, C27.1, C28.1, C29.1, C30.1, C32.1, C34.2, C36.2, C38.2, C4.2, C6.2, C7.-, Q1.GND, R100.1, R103.1, R104.2, R30.1, R35.1, R4.2, R42.2, R43.1, R6.2, R8.2, RT2.2, U$1.AGND, U$1.PGND, U$5.GND, U1.S, U1.S_2, U1.S_3, U11.S, U11.S_2, U11.S_3, U12.GND, U12.PFM_PWM, U12.PGND_2, U12.PGND_3, U15.DVSS, U15.VSS_QFN, U2.S, U2.S_2, U2.S_3, U3.S, U3.S_2, U3.S_3, U7.PFM_PWM, U7.PGND, U7.PGND_2, U7.PGND_3, U8.GND1, U8.GND2, U8.GND3, U8.GND4, U8.GND5, U9.EPAD, U9.GND, U9.TERM_EN
- net HEAT1: now also Q1.D, Q1.D_2, Q1.D_3, Q1.D_4; no longer U1.D, U1.D_2, U1.D_3, U1.D_4
- net HEAT2: now also Q2.D, Q2.D_2, Q2.D_3, Q2.D_4; no longer U2.D, U2.D_2, U2.D_3, U2.D_4
- net HEAT3: now also Q3.D, Q3.D_2, Q3.D_3, Q3.D_4; no longer U3.D, U3.D_2, U3.D_3, U3.D_4
- net I2C_SCL: now also U1.P1.7/TB0.4/UCB0SOMI/UCB0SCL/TA1.0; no longer U15.P1.7/TB0.4/UCB0SOMI/UCB0SCL/TA1.0
- net I2C_SDA: now also U1.P1.6/TB0.3/UCB0SIMO/UCB0SDA/TA0.0; no longer U15.P1.6/TB0.3/UCB0SIMO/UCB0SDA/TA0.0
- net IND: now also L5.2, U7.SW; no longer L3.2, U8.SW
- net I_IN: now also C9.2, R22.1, U1.P1.1/TA0.2/A1/C1; no longer C8.2, R25.1, U15.P1.1/TA0.2/A1/C1
- net I_OUT: now also C10.2, R24.1, U1.P1.0/TA0.1/A0/C0; no longer C9.2, R26.1, U15.P1.0/TA0.1/A0/C0
- net LED5: now also R14.2; no longer R15.2
- net N$1: now also L3.1, U6.L1, U6.L1_2, U6.L1_3; no longer L2.1, U12.L1, U12.L1_2, U12.L1_3
- net N$10: now also Q7G$1.G, U11.OUT; no longer Q2G$1.G, U$5.OUT
- net N$11: now also L1.1, U4.L1, U4.L1_2, U4.L1_3; no longer L100.1, U7.L1, U7.L1_2, U7.L1_3
- net N$12: now also L1.2, U4.L2, U4.L2_2, U4.L2_3; no longer L100.2, U7.L2, U7.L2_2, U7.L2_3
- net N$13: now also JP1.1, R1.1, U1.RST/SBWTDIO; no longer JP2.1, R19.1, U15.RST/SBWTDIO
- net N$14: now also R14.1; no longer R15.1
- net N$15: now also JP1.2, U1.TEST/SBWTCK; no longer JP2.2, U15.TEST/SBWTCK
- net N$16: now also C7.2, U1.LFXOUT, X1.1; no longer C39.2, Q1.1, U15.LFXOUT
- net N$17: now also C6.2, U1.LFXIN, X1.2; no longer C40.2, Q1.2, U15.LFXIN
- net N$18: now also U1.P2.1/TB0.0/UCA0RXD/UCA0SOMI; no longer U15.P2.1/TB0.0/UCA0RXD/UCA0SOMI
- net N$19: now also R4.1, R5.2, U2A.OUT; no longer IC1A.OUT, R1.2, R9.1
- net N$2: now also R37.1, U7.PG; no longer R28.1, U8.PG
- net N$20: now also R2.1, R4.2, U2A.-IN; no longer IC1A.-IN, R10.1, R9.2
- net N$21: now also R3.2, U2A.+IN; no longer IC1A.+IN, R21.2
- net N$22: now also R7.2, R8.1, U2B.OUT; no longer IC1B.OUT, R17.1, R2.2
- net N$23: now also R8.2, R9.1, U2B.-IN; no longer IC1B.-IN, R17.2, R18.1
- net N$24: now also R25.1, R6.2, U2B.+IN; no longer IC1B.+IN, R20.2, R22.1
- net N$25: now also R24.2, U10.OUT; no longer R26.2, U$3.OUT
- net N$26: now also R22.2, U9.OUT; no longer R25.2, U$2.OUT
- net N$27: now also Q3.G, R20.1; no longer R7.1, U3.G
- net N$28: now also U1.P2.0/TB0.6/UCA0TXD/UCA0SIMO; no longer U15.P2.0/TB0.6/UCA0TXD/UCA0SIMO
- net N$29: now also U1.P2.3/TA0.0/UCA1STE/A6; no longer U15.P2.3/TA0.0/UCA1STE/A6
- net N$3: now also L3.2, U6.L2, U6.L2_2, U6.L2_3; no longer L2.2, U12.L2, U12.L2_2, U12.L2_3
- net N$30: now also U1.P2.4/TA1.0/UCA1CLK/A7; no longer U15.P2.4/TA1.0/UCA1CLK/A7
- net N$31: now also Q2.G, R18.1; no longer R5.1, U2.G
- net N$32: now also U10.IN+; no longer U$3.IN+
- net N$33: now also U10.IN-; no longer U$3.IN-
- net N$34: now also U9.IN+; no longer U$2.IN+
- net N$35: now also U9.IN-; no longer U$2.IN-
- net N$36: now also U1.P2.6/TB0.1/UCA1RXD/UCA1SOMI; no longer U15.P2.6/TB0.1/UCA1RXD/UCA1SOMI
- net N$37: now also Q1.G, R16.1; no longer R3.1, U1.G
- net N$38: now also C32.2, U12.BOOT; no longer C31.2, U$1.BOOT
- net N$39: now also R11.2; no longer R12.2
- net N$4: now also L4.2; no longer 6.8UH.2
- net N$40: now also R11.1; no longer R12.1
- net N$41: now also U1.P2.5/TB0.0/UCA1TXD/UCA1SIMO; no longer U15.P2.5/TB0.0/UCA1TXD/UCA1SIMO
- net N$42: now also C27.1, R39.1; no longer C22.1, R41.1
- net N$43: now also R10.2; no longer R11.2
- net N$45: now also R10.1; no longer R11.1
- net N$46: now also R13.2; no longer R14.2
- net N$47: now also R13.1; no longer R14.1
- net N$48: now also R15.2; no longer R16.2
- net N$49: now also R15.1; no longer R16.1
- net N$5: now also C20.1, U7.SS; no longer C13.1, U8.SS
- net N$50: now also C32.1, L6.2, R43.2, U12.SW1, U12.SW2, U12.SW3, U12.SW4; no longer C31.1, L4.2, R39.2, U$1.SW1, U$1.SW2, U$1.SW3, U$1.SW4
- net N$51: now also R12.2; no longer R13.2
- net N$52: now also R12.1; no longer R13.1
- net N$53: now also R43.1, U12.FSW; no longer R39.1, U$1.FSW
- net N$54: now also C37.1, R45.1; no longer C25.1, R37.1
- net N$56: now also C46.1, U12.SS; no longer C36.1, U$1.SS
- net N$57: now also R44.2, U12.ILIM; no longer R35.2, U$1.ILIM
- net N$58: now also C35.1, R45.2, U12.COMP; no longer C24.1, R37.2, U$1.COMP
- net N$59: now also C33.1, U12.VCC; no longer C23.1, U$1.VCC
- net N$6: now also L2.1, U8.L1, U8.L1_2, U8.L1_3; no longer L1.1, U6.L1, U6.L1_2, U6.L1_3
- net N$60: now also R46.2, R47.1, U12.FB; no longer R36.2, R38.1, U$1.FB
- net N$64: now also R29.1, R33.2, U5.MPPSET; no longer R100.2, R101.1, U9.MPPSET
- net N$69: now also R30.1; no longer R29.1
- net N$7: now also L2.2, U8.L2, U8.L2_2, U8.L2_3; no longer L1.2, U6.L2, U6.L2_2, U6.L2_3
- net N$70: now also U5.STAT2; no longer U9.STAT2
- net N$71: now also U5.STAT1; no longer U9.STAT1
- net N$72: now also C18.1, RT3.1, U5.VREF; no longer C20.1, RT1.1, U9.VREF
- net N$73: now also C28.1, U5.VCC; no longer C21.1, U9.VCC
- net N$76: now also C29.1, L4.1, Q5.S, Q5.S_2, Q5.S_3, Q6.D, Q6.D_2, Q6.D_3, Q6.D_4, U5.PH; no longer 6.8UH.1, C100.1, U10.S, U10.S_2, U10.S_3, U11.D, U11.D_2, U11.D_3, U11.D_4, U9.PH
- net N$77: now also C17.2, U5.SRP; no longer C15.2, U9.SRP
- net N$78: now also C17.1, U5.SRN; no longer C15.1, U9.SRN
- net N$80: now also Q5.G, U5.HIDRV; no longer U10.G, U9.HIDRV
- net N$81: now also Q6.G, U5.LODRV; no longer U11.G, U9.LODRV
- net N$82: now also C30.2, R34.2, R35.1, R41.1, U5.VFB; no longer C26.2, R32.1, R33.2, R34.1, U9.VFB
- net N$84: now also C16.1, U5.REGN; no longer C101.1, U9.REGN
- net N$85: now also C29.2, U5.BTST; no longer C100.2, U9.BTST
- net N$9: now also R48.1, U12.MODE; no longer R42.1, U$1.MODE
- net SC+: now also C40.2, Q5.D, Q5.D_2, Q5.D_3, Q5.D_4, R25.2, R28.2, R30.2, R39.2; no longer C32.2, R101.2, R102.2, R22.2, R41.2, U10.D, U10.D_2, U10.D_3, U10.D_4
- net SC_OUT: now also C30.1, C41.1, C42.1, R35.2, R41.2; no longer C26.1, C37.1, C38.1, R32.2, R34.2
- net TS: now also RT3.2, RT4.1, U5.TS; no longer RT1.2, RT2.1, U9.TS
- net V_BAT: now also R5.1, U1.P1.3/TA1.2/UCB0STE/A3/C3; no longer R1.1, U15.P1.3/TA1.2/UCB0STE/A3/C3
- net V_SC: now also C3.2, R7.1, U1.P1.2/TA1.1/A2/C2; no longer C2.2, R2.1, U15.P1.2/TA1.1/A2/C2
Other:
- moved on the sheet: C10, C11, C12, C13, C14, C15, C16, C17, C18, C19, C2, C20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

Commit message: adjusted final resistor values for eps v1.0
Parts:
- C28: value 1u -> 1uF
- R2, R23: value 200k -> 200k (0.1%)
- R25, R9: value 200k -> 330k (0.1%)
- R28: value 1M -> dnp
- R29: value (none) -> Rmpph
- R3, R4, R6, R8: value 100k -> 100k (0.1%)
- R33: value (none) -> Rmppl
- R34, R35: value 100k -> 100k (1%)
- R41: value 2.2M -> 2.2M (1%)
- R47: value 470k -> 456k
- RS2, RS3: value 50m -> 10m
- RT3: value 2723 -> 2696
- RT4: value 8501 -> 8187
- RTH: value (none) -> 103AT
Connections:
- net A4_EXT renamed A_EXT0
- removed net A5_EXT: JP2.9, RT1.2, U1.P1.5/TB0.2/UCA0CLK/A5/C5
- new net A_EXT5: JP2.1, U1.P4.3/A11
- net A_EXT1: now also JP2.9, RT1.2, U1.P1.5/TB0.2/UCA0CLK/A5/C5; no longer JP2.7, U1.P4.0/A8
- net A_EXT2: now also JP2.7, U1.P4.0/A8; no longer JP2.5, U1.P4.1/A9
- net A_EXT3: now also JP2.5, U1.P4.1/A9; no longer JP2.3, U1.P4.2/A10
- net A_EXT4: now also JP2.3, U1.P4.2/A10; no longer JP2.1, U1.P4.3/A11
Other:
- note added: "-25°C - 60°C charge range (see BOM for calculation)"
- note added: "-> Vout = 11.0 V"
- note added: "470kOhm for R47 for Vout = 11.4V"
- note added: "input range: 0 - 5V"
- note added: "input range: 0 - 8.5V"
- note removed: "-> Vout = 11.4 V"
- note removed: "456kOhm for R23 for Vout = 11V"
- moved on the sheet: C30, R34, R35
